File: pilkbrain.kicad_pcb (KiCad board)
At the start: 4 copper layers, 33.2 x 21 mm, 102 parts, among them SW2 EVQPUC02K, SW3 EVQPUC02K, U1 ESP32-C3, U10 TS5A23157DGSR, U12 ESP32-S3, U3 SPX3819M5-L-3-3, U4 BQ24073RGT, U6 W25Q128JVS, U7 MT9700, U8 MAX98357AEWL+T, U9 MT9700, Y1 XO-40M, Y2 XO-32K

Commit message: before route
Parts:
- removed C10, C22: 10u, Capacitor_SMD:C_0603_1608Metric
- removed C25, C3: 100n, Capacitor_SMD:C_0402_1005Metric
- removed H1, H2, H3: M2, MountingHole:MountingHole_2.2mm_M2
- removed PAD16: BAT+, Critbit_lib:diy_castellate_2.54
- removed R12, R20, R26, R27, R28, R29: DNP/0603, Resistor_SMD:R_0603_1608Metric
- removed R21, R22, R23, R25: 0R/0603, Resistor_SMD:R_0603_1608Metric
- removed R30: 3k3/0603, Resistor_SMD:R_0603_1608Metric
- removed REF**: TF-SMD_TF-123-ARP9H15, easyeda2kicad:TF-SMD_TF-123-ARP9H15
- removed U10: TS5A23157DGSR, easyeda2kicad:MSOP-10_L3.0-W3.0-P0.50-LS5.0-BL
- removed U12: ESP32-S3, Package_DFN_QFN:QFN-56-1EP_7x7mm_P0.4mm_EP4x4mm
- removed U6: W25Q128JVS, Package_SO:SOIC-8_5.23x5.23mm_P1.27mm
- added C26: 1u, Capacitor_SMD:C_0402_1005Metric, B.Cu at (111.6, 42.2)
- added C27: 100n, Capacitor_SMD:C_0402_1005Metric, B.Cu at (109.8, 51.7)
- added C29: 1u, Capacitor_SMD:C_0402_1005Metric, B.Cu at (114.1, 50.5)
- added C30: 100n, Capacitor_SMD:C_0402_1005Metric, B.Cu at (114.1, 49.5)
- added C31: 100n, Capacitor_SMD:C_0402_1005Metric, B.Cu at (115.6, 44.3)
- added J1: USB_C_Receptacle_USB2.0, Connector_USB:USB_C_Receptacle_HRO_TYPE-C-31-M-12, B.Cu at (88.5, 54.5)
- added J2: Conn_01x05, Connector_PinHeader_1.27mm:PinHeader_1x05_P1.27mm_Vertical, F.Cu at (115.4, 42.6)
- added PAD21: BAT-, Critbit_lib:diy_castellate_2.54, B.Cu at (119.8, 61.8)
- added PAD22: BAT-, Critbit_lib:diy_castellate_2.54, B.Cu at (121.8, 61.8)
- added PAD23: BAT-, Critbit_lib:diy_castellate_2.54, B.Cu at (123.8, 61.8)
- added PAD24: BAT-, Critbit_lib:diy_castellate_2.54, B.Cu at (109.4, 39.5)
- added PAD25: BAT-, Critbit_lib:diy_castellate_2.54, B.Cu at (106.9, 39.5)
- added PAD26: BAT-, Critbit_lib:diy_castellate_2.54, B.Cu at (104.4, 39.5)
- added R31: 10k, Resistor_SMD:R_0402_1005Metric, B.Cu at (107.9, 51.7)
- added R32: 10k, Resistor_SMD:R_0402_1005Metric, B.Cu at (111.6, 51.7)
- added R33: 10k, Resistor_SMD:R_0402_1005Metric, B.Cu at (113.5, 51.7)
- added R34: 10k, Resistor_SMD:R_0402_1005Metric, B.Cu at (115.4, 51.8)
- added R35: 100k, Resistor_SMD:R_0402_1005Metric, B.Cu at (103.4, 52.9)
- added R36: 5.1k, Resistor_SMD:R_0402_1005Metric, B.Cu at (90.5, 48.8)
- added R37: 5.1k, Resistor_SMD:R_0402_1005Metric, B.Cu at (88.6, 48.8)
- added R6: 10k, Resistor_SMD:R_0402_1005Metric, B.Cu at (106.0, 51.7)
- added U13: ESP32-S3, Package_DFN_QFN:QFN-56-1EP_7x7mm_P0.4mm_EP4x4mm, B.Cu at (109.0, 46.9)
- C1: value 100n -> 10n
- C20: value 10u -> 1u; footprint Capacitor_SMD:C_0603_1608Metric -> Capacitor_SMD:C_0402_1005Metric
- C23: value 10u -> 100n; footprint Capacitor_SMD:C_0603_1608Metric -> Capacitor_SMD:C_0402_1005Metric
- R1: value 1k/0603 -> 3k3; footprint Resistor_SMD:R_0603_1608Metric -> Resistor_SMD:R_0402_1005Metric
- R2: value 100 -> 10k
- R4: value 3k3/0603 -> 3k3; footprint Resistor_SMD:R_0603_1608Metric -> Resistor_SMD:R_0402_1005Metric
- U1: value ESP32-C3 -> TF-123-ARP9H17; footprint Package_DFN_QFN:QFN-32-1EP_5x5mm_P0.5mm_EP3.45x3.45mm -> easyeda2kicad:TF-SMD_TF-123-ARP9H15
- U2: moved to B.Cu
- U5: footprint Critbit_lib:OLED_4Pin_128x32 -> Critbit_lib:OLED_4Pin_128x64_new; moved to B.Cu
- moved U2 155.5 mm to (100.3, 135.4), turned to 0 degrees
- moved U5 102.1 mm to (126.9, 146.3), turned to 0 degrees
- moved R4 53.6 mm to (116.0, 59.1), turned to 90 degrees
- moved PAD4 37.4 mm to (124.0, 39.5), turned to -90 degrees
- moved PAD3 34.2 mm to (122.0, 39.5), turned to -90 degrees
- moved PAD20 24.1 mm to (113.8, 61.9), turned to 90 degrees
- moved PAD1 23.6 mm to (96.4, 61.9)
- moved PAD2 23.6 mm to (100.4, 61.9)
- moved PAD5 23.6 mm to (98.4, 61.9)
- moved R15 23.5 mm to (96.5, 59.4), turned to 0 degrees
- moved PAD17 23.1 mm to (111.7, 39.5), turned to -90 degrees
- moved U9 22.8 mm to (119.0, 56.5)
- moved R18 22.7 mm to (118.3, 54.3), turned to 0 degrees
- moved PAD15 22.7 mm to (116.3, 39.5), turned to -90 degrees
- moved PAD14 22.5 mm to (114.0, 39.5), turned to -90 degrees
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Connections:
- C18 pad 1: Net-(C18-Pad1) -> /BUT2
- C20 pad 1: Net-(U1-VDD_SPI/GPIO11) -> +3.3V
- C23 pad 1: Net-(C23-Pad1) -> VDD3P3
- C35 pad 1: Net-(U1-LNA_IN) -> Net-(U13-LNA_IN/RF)
- C5 pad 1: Net-(U1-XTAL_32K_P/ADC1_CH0) -> Net-(U13-GPIO15/ADC2_CH4/XTAL_32K_P)
- C6 pad 1: Net-(U1-XTAL_32K_N/ADC1_CH1) -> Net-(U13-GPIO16/ADC2_CH5/XTAL_32K_N)
- C7 pad 1: Net-(U1-XTAL_P) -> Net-(U13-XTAL_P)
- C8 pad 1: Net-(U1-XTAL_N) -> Net-(U13-XTAL_N)
- L1 pad 2: Net-(C23-Pad1) -> VDD3P3
- L2 pad 2: Net-(U1-LNA_IN) -> Net-(U13-LNA_IN/RF)
- PAD14 pad 1: /TARG_TX_B2 -> /TARG_TX
- PAD15 pad 1: /TARG_RX_LRCLK -> /TARG_RX
- PAD19 pad 1: Net-(PAD19-Pad1) -> /3V3_OUT
- PAD20 pad 1: Net-(PAD20-Pad1) -> GND
- PAD8 pad 1: Net-(PAD8-Pad1) -> /I2C_SCL
- PAD9 pad 1: Net-(PAD9-Pad1) -> /I2C_SDA
- R1 pad 1: Net-(C18-Pad1) -> /I2C_SDA
- R1 pad 2: /TARG_TX_B2 -> +3.3V
- R19 pad 1: Net-(C18-Pad1) -> /BUT2
- R2 pad 1: /I2S_LRCLK -> /SD_DAT1
- R2 pad 2: /TARG_RX_LRCLK -> +3.3V
- SW2 pad 2: Net-(C18-Pad1) -> /BUT2
- SW2 pad 4: Net-(C18-Pad1) -> /BUT2
- U1 pad 1: Net-(U1-LNA_IN) -> /SD_DAT2
- U1 pad 10: /EN_RIGHT -> unconnected-(U1-Pad10)
- U1 pad 11: +3.3V -> unconnected-(U1-Pad11)
- U1 pad 12: /I2S_DAT -> unconnected-(U1-Pad12)
- U1 pad 13: /I2S_CLK -> unconnected-(U1-Pad13)
- U1 pad 2: Net-(C23-Pad1) -> /SD_DAT3
- U1 pad 3: Net-(C23-Pad1) -> /SD_CMD
- U1 pad 4: Net-(U1-XTAL_32K_P/ADC1_CH0) -> +3.3V
- U1 pad 5: Net-(U1-XTAL_32K_N/ADC1_CH1) -> /SD_CLK
- U1 pad 6: /I2C_SCL -> GND
- U1 pad 7: /ESP_EN -> /SD_DAT0
- U1 pad 8: /I2C_SDA -> /SD_DAT1
- U1 pad 9: /EN_LEFT -> Net-(U1-SWITCH)
- Y1 pad 1: Net-(U1-XTAL_P) -> Net-(U13-XTAL_P)
- Y1 pad 3: Net-(U1-XTAL_N) -> Net-(U13-XTAL_N)
- Y2 pad 1: Net-(U1-XTAL_32K_P/ADC1_CH0) -> Net-(U13-GPIO15/ADC2_CH4/XTAL_32K_P)
- Y2 pad 2: Net-(U1-XTAL_32K_N/ADC1_CH1) -> Net-(U13-GPIO16/ADC2_CH5/XTAL_32K_N)
Routing:
- net Net-(C23-Pad1): track 11.6 -> 0.00 mm, vias 2 -> 0
- net (no net): track 0.00 -> 9.25 mm
- net Net-(U1-SPICS0/GPIO14): track 9.20 -> 0.00 mm, vias 2 -> 0
- net +3.3V: track 9.07 -> 0.00 mm, vias 1 -> 0
- net Net-(U1-SPICLK/GPIO15): track 8.08 -> 0.00 mm
- net Net-(U1-SPIHD/GPIO12): track 6.75 -> 0.00 mm, vias 2 -> 0
- net /ESP_EN: track 6.61 -> 0.00 mm, vias 1 -> 0
- net Net-(U1-SPIWP/GPIO13): track 6.30 -> 0.00 mm, vias 2 -> 0
- net Net-(U1-VDD_SPI/GPIO11): track 6.01 -> 0.00 mm
- net Net-(U1-XTAL_N): track 5.34 -> 0.00 mm
- net /EN_PERIPH: track 5.17 -> 0.00 mm
- net Net-(U1-XTAL_32K_N/ADC1_CH1): track 4.83 -> 0.00 mm
- net GND: track 6.09 -> 1.50 mm, vias 3 -> 2
- net /TARG_RX_LRCLK: track 4.25 -> 0.00 mm, vias 1 -> 0
- net Net-(U1-SPIQ/GPIO17): track 3.98 -> 0.00 mm, vias 2 -> 0
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Other:
- board size 33.2 x 21 mm -> 38.8 x 24.5 mm
- board text added: "1"
- board text added: "CHG"
- board text added: "Pilkbrain 10.24 @cb t"
- board text added: "VIN"

Commit message: before move 4L
Parts:
- removed R15: 10k/0603, Resistor_SMD:R_0603_1608Metric
- added R12: 10k, Resistor_SMD:R_0402_1005Metric, B.Cu at (96.4, 59.4)
- added REF**: MountingHole_2.2mm_M2, MountingHole:MountingHole_2.2mm_M2, F.Cu at (123.2, 51.0)
- moved D4 11.9 mm to (102.1, 57.1), turned to -90 degrees
- moved R9 8.45 mm to (101.8, 55.0)
- moved R19 5.91 mm to (120.6, 44.3), turned to 180 degrees
- moved C18 5.82 mm to (119.1, 44.6)
- moved C13 5.59 mm to (102.9, 51.8), turned to 90 degrees
- moved C34 3.67 mm to (100.2, 42.1), turned to -90 degrees
- moved R13 3.51 mm to (97.5, 47.0), turned to 0 degrees
- moved R8 2.97 mm to (99.6, 48.1), turned to 90 degrees
- moved R2 1.75 mm to (104.4, 50.0), turned to 90 degrees
- moved L2 1.70 mm to (102.2, 41.5)
- moved C20 1.69 mm to (103.4, 42.5)
- moved C7 1.53 mm to (103.4, 44.9)
- moved C1 1.49 mm to (103.4, 43.7)
- moved R34 1.38 mm to (114.3, 52.7)
- moved R7 1.20 mm to (101.2, 43.7), turned to 180 degrees
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Connections:
- PAD14 pad 1: /TARG_TX -> unconnected-(PAD14-Pad1)
- PAD15 pad 1: /TARG_RX -> unconnected-(PAD15-Pad1)
- PAD17 pad 1: /BOOT_BUT1 -> unconnected-(PAD17-Pad1)
- R1 pad 2: +3.3V -> /3V3_OUT
- R4 pad 2: +3.3V -> /3V3_OUT
- U13 pad 10: /I2S_LRCLK -> unconnected-(U13-GPIO5/ADC1_CH4-Pad10)
- U13 pad 11: /I2S_DAT -> unconnected-(U13-GPIO6/ADC1_CH5-Pad11)
- U13 pad 12: /I2S_CLK -> unconnected-(U13-GPIO7/ADC1_CH6-Pad12)
- U13 pad 15: /EN_PERIPH -> unconnected-(U13-GPIO10/ADC1_CH9-Pad15)
- U13 pad 16: unconnected-(U13-GPIO11/ADC2_CH0-Pad16) -> /I2S_CLK
- U13 pad 17: unconnected-(U13-GPIO12/ADC2_CH1-Pad17) -> /I2S_DAT
- U13 pad 18: unconnected-(U13-GPIO13/ADC2_CH2-Pad18) -> /I2S_LRCLK
- U13 pad 23: unconnected-(U13-GPIO17/ADC2_CH6-Pad23) -> /EN_PERIPH
- U13 pad 24: unconnected-(U13-GPIO18/ADC2_CH7-Pad24) -> /SD_DAT3
- U13 pad 27: unconnected-(U13-GPIO21-Pad27) -> /SD_CMD
- U13 pad 36: unconnected-(U13-SPICLK_N/GPIO48-Pad36) -> /SD_DAT2
- U13 pad 37: unconnected-(U13-SPICLK_P/GPIO47-Pad37) -> /WS2812_OUT
- U13 pad 39: unconnected-(U13-GPIO34-Pad39) -> /SD_CLK
- U13 pad 40: unconnected-(U13-GPIO35-Pad40) -> /I2C_SCL
- U13 pad 41: unconnected-(U13-GPIO36-Pad41) -> /SD_DAT0
- U13 pad 42: unconnected-(U13-GPIO37-Pad42) -> /I2C_SDA
- U13 pad 43: unconnected-(U13-GPIO38-Pad43) -> /SD_DAT1
- U13 pad 7: /I2C_SCL -> unconnected-(U13-GPIO2/ADC1_CH1-Pad7)
- U13 pad 8: /I2C_SDA -> unconnected-(U13-GPIO3/ADC1_CH2-Pad8)
Routing:
- net GND: track 1.50 -> 89.2 mm, vias 2 -> 29
- net +3.3V: track 0.00 -> 75.5 mm, vias 0 -> 13
- net +4V: track 0.00 -> 34.8 mm, vias 0 -> 2
- net /USBDM: track 0.00 -> 24.7 mm, vias 0 -> 1
- net /USBDP: track 0.00 -> 24.5 mm, vias 0 -> 1
- net /I2C_SDA: track 0.00 -> 22.5 mm, vias 0 -> 3
- net /WS2812_OUT: track 0.00 -> 21.8 mm, vias 0 -> 3
- net /BOOT_BUT1: track 0.00 -> 20.2 mm, vias 0 -> 1
- net /I2C_SCL: track 0.00 -> 19.4 mm, vias 0 -> 2
- net /ESP_EN: track 0.00 -> 17.9 mm, vias 0 -> 3
- net /LIPO+: track 0.00 -> 13.3 mm, vias 0 -> 1
- net /I2S_LRCLK: track 0.00 -> 11.6 mm, vias 0 -> 2
- net /EN_PERIPH: track 0.00 -> 11.3 mm
- net /WS2812_VDD: track 1.24 -> 10.8 mm
- net Net-(U8-OUTP): track 0.25 -> 9.55 mm
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- added copper zone on F.Cu, net +3.3V
- added copper zone on F.Cu, net GND
Other:
- copper layers 4 -> 2
- board text removed: "1"
- board text removed: "Pilkbrain 10.24 @cb t"

Commit message: DRC
Parts:
- removed C31: 100n, Capacitor_SMD:C_0402_1005Metric
- removed REF**: MountingHole_2.2mm_M2, MountingHole:MountingHole_2.2mm_M2
- added H1: M2, MountingHole:MountingHole_2.2mm_M2, F.Cu at (123.0, 50.8)
- moved R5 6.75 mm to (118.4, 47.2), turned to 0 degrees
- moved R3 6.62 mm to (120.3, 47.2), turned to 0 degrees
- moved R19 5.01 mm to (115.6, 43.9)
- moved R24 4.70 mm to (118.7, 53.7), turned to -90 degrees
- moved C18 3.51 mm to (115.6, 44.9), turned to 0 degrees
- moved C19 3.06 mm to (120.1, 54.2), turned to 0 degrees
- moved C6 3.00 mm to (117.7, 48.6), turned to 90 degrees
- moved C33 2.78 mm to (120.6, 44.7), turned to 90 degrees
- moved R16 2.15 mm to (120.2, 46.1), turned to 0 degrees
- moved R10 1.78 mm to (120.1, 53.2)
- moved U8 1.77 mm to (119.3, 44.4), turned to -90 degrees
- moved C17 1.51 mm to (117.8, 45.8), turned to -90 degrees
- moved R8 1.49 mm to (98.6, 47.0), turned to 180 degrees
- moved C5 1.10 mm to (114.3, 46.8), turned to -90 degrees
- moved R18 0.85 mm to (117.7, 53.7), turned to -90 degrees
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Connections:
- PAD14 pad 1: unconnected-(PAD14-Pad1) -> /EXTIO_3
- PAD15 pad 1: unconnected-(PAD15-Pad1) -> /EXTIO_2
- PAD17 pad 1: unconnected-(PAD17-Pad1) -> GND
- PAD18 pad 1: GND -> /EXTIO_1
- PAD24 pad 1: unconnected-(PAD24-Pad1) -> /EXTIO_4
- PAD25 pad 1: unconnected-(PAD25-Pad1) -> /EXTIO_5
- PAD26 pad 1: unconnected-(PAD26-Pad1) -> /EXTIO_6
- R18 pad 2: Net-(U9-EN) -> /EN_3V3OUT
- U13 pad 10: unconnected-(U13-GPIO5/ADC1_CH4-Pad10) -> /EXTIO_2
- U13 pad 13: /WS2812_OUT -> /BUT2
- U13 pad 14: unconnected-(U13-GPIO9/ADC1_CH8-Pad14) -> /EXTIO_1
- U13 pad 15: unconnected-(U13-GPIO10/ADC1_CH9-Pad15) -> /VBAT_MEAS
- U13 pad 16: /I2S_CLK -> /I2S_LRCLK
- U13 pad 18: /I2S_LRCLK -> /I2S_CLK
- U13 pad 19: unconnected-(U13-GPIO14/ADC2_CH3-Pad19) -> /EN_3V3OUT
- U13 pad 6: unconnected-(U13-GPIO1/ADC1_CH0-Pad6) -> /EXTIO_6
- U13 pad 7: unconnected-(U13-GPIO2/ADC1_CH1-Pad7) -> /EXTIO_5
- U13 pad 8: unconnected-(U13-GPIO3/ADC1_CH2-Pad8) -> /EXTIO_4
- U13 pad 9: unconnected-(U13-GPIO4/ADC1_CH3-Pad9) -> /EXTIO_3
- U9 pad 4: Net-(U9-EN) -> /EN_3V3OUT
Routing:
- net /BUT2: track 8.49 -> 34.1 mm, vias 0 -> 3
- net /BOOT_BUT1: track 20.2 -> 42.2 mm, vias 1 -> 2
- net +3.3V: track 75.5 -> 56.7 mm, vias 13 -> 16
- net /TARG_RX: track 0.00 -> 18.4 mm, vias 0 -> 1
- net /EN_3V3OUT: track 0.00 -> 17.1 mm, vias 0 -> 2
- net /TARG_TX: track 0.00 -> 16.3 mm, vias 0 -> 1
- net Net-(U4-TS): track 3.12 -> 15.5 mm, vias 0 -> 1
- net Net-(J1-CC1): track 0.00 -> 10.4 mm, vias 0 -> 2
- net VBUS: track 5.67 -> 15.7 mm
- net /VBAT_MEAS: track 1.00 -> 10.7 mm
- net /EXTIO_1: track 0.00 -> 9.46 mm, vias 0 -> 1
- net /LIPO+: track 13.3 -> 3.91 mm, vias 1 -> 2
- net /EXTIO_2: track 0.00 -> 9.31 mm, vias 0 -> 2
- net /BQ_PGOOD: track 0.99 -> 9.20 mm, vias 1 -> 2
- net /USBDP: track 24.5 -> 32.3 mm, vias 1 -> 2
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- added copper zone on In2.Cu, net +3.3V
- added copper zone on B.Cu, net +4V
- added copper zone on F.Cu, net +4V
- added copper zone on In2.Cu, net /3V3_OUT
- added copper zone on In2.Cu, net /LIPO+
- added copper zone on In2.Cu, net /WS2812_VDD
- added copper zone on In1.Cu, net GND
- removed copper zone on F.Cu, net +3.3V
- removed copper zone on F.Cu, net GND
Other:
- copper layers 2 -> 4

Commit message: before fab out
Parts:
- removed U2: ~, Critbit_lib:OLED_4Pin_64x48
- removed U5: ~, Critbit_lib:OLED_4Pin_128x64_new
- added C3: 1u, Capacitor_SMD:C_0402_1005Metric, B.Cu at (103.0, 49.6)
- added D1: LED_WHITE, LED_SMD:LED_0603_1608Metric, B.Cu at (97.5, 45.3)
- added L3: 24nH, Inductor_SMD:L_0402_1005Metric, B.Cu at (103.2, 45.1)
- added PAD16: 7, Critbit_lib:diy_castellate_2.54, B.Cu at (104.7, 39.5)
- added PAD27: 8, Critbit_lib:diy_castellate_2.54, B.Cu at (102.7, 39.5)
- added PAD28: 9, Critbit_lib:diy_castellate_2.54, B.Cu at (94.5, 48.4)
- added PAD29: 10, Critbit_lib:diy_castellate_2.54, B.Cu at (94.5, 50.4)
- added R15: 10k, Resistor_SMD:R_0402_1005Metric, B.Cu at (101.7, 44.1)
- C1: value 10n -> 100n
- C21: value 100n -> 1u
- C34, C35: value 100n -> 3.3p
- C5, C6, C7, C8: value 20p(TBD) -> 12p
- L1: value 2nH -> 2nH/500mA
- L2: value TBD -> 2nH/500mA
- PAD11: value BAT- -> EN_3V3
- PAD12: value BAT- -> 5V
- PAD13: value BAT- -> GND; moved to B.Cu
- PAD14: value BAT+ -> 3; moved to F.Cu
- PAD15: value BAT+ -> 2; moved to F.Cu
- PAD17: value BAT+ -> GND
- PAD18: value BAT+ -> 1
- PAD19: value BAT- -> 3V3_OUT
- PAD20, PAD23: value BAT- -> GND
- PAD21: value BAT- -> 4V_OUT
- PAD22: value BAT- -> WS2812_OUT
- PAD24: value BAT- -> 4; moved to F.Cu
- PAD25: value BAT- -> 5; moved to F.Cu
- PAD26: value BAT- -> 6; moved to F.Cu
- PAD6: value BAT- -> DM
- PAD7: value BAT- -> DP
- PAD8: value BAT- -> SCL
- PAD9: value BAT- -> SDA
- R1, R4: value 3k3 -> 2k
- R13, R14: value 3k -> 2k
- moved C21 15.7 mm to (116.9, 43.7)
- moved R7 14.3 mm to (115.5, 44.2), turned to -90 degrees
- moved C19 5.95 mm to (118.1, 59.8), turned to 180 degrees
- moved C18 5.70 mm to (120.3, 48.1)
- moved R24 5.35 mm to (120.6, 58.7), turned to 90 degrees
- moved R19 4.87 mm to (118.1, 48.1)
- moved R35 3.74 mm to (102.0, 55.0), turned to 0 degrees
- moved R2 2.92 mm to (104.1, 52.9), turned to -90 degrees
- moved R13 2.86 mm to (99.5, 46.2), turned to -90 degrees
- moved PAD26 2.30 mm to (106.7, 39.5)
- moved J1 2.20 mm to (88.5, 56.7)
- moved PAD12 2.20 mm to (94.5, 53.5)
- moved PAD13 2.20 mm to (94.5, 59.5)
- moved PAD6 2.20 mm to (94.5, 55.5)
- moved PAD7 2.20 mm to (94.5, 57.5)
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Connections:
- C7 pad 1: Net-(U13-XTAL_P) -> Net-(C7-Pad1)
- D3 pad 2: +4V -> +3.3V
- D4 pad 2: +4V -> +3.3V
- PAD10 pad 1: /EN_LEFT -> /EN_PERIPH
- PAD11 pad 1: /EN_RIGHT -> /EN_3V3OUT
- U13 pad 44: unconnected-(U13-MTCK/JTAG/GPIO39-Pad44) -> /EXTIO_10
- U13 pad 45: unconnected-(U13-MTDO/JTAG/GPIO40-Pad45) -> /EXTIO_8
- U13 pad 47: unconnected-(U13-MTDI/JTAG/GPIO41-Pad47) -> /EXTIO_7
- U13 pad 48: unconnected-(U13-MTMS/JTAG/GPIO42-Pad48) -> /EXTIO_9
- U13 pad 51: unconnected-(U13-GPIO45-Pad51) -> /BQ_PGOOD
- U13 pad 52: unconnected-(U13-GPIO46-Pad52) -> /LED_STA
- U3 pad 3: unconnected-(U3-EN-Pad3) -> +4V
- Y1 pad 1: Net-(U13-XTAL_P) -> Net-(C7-Pad1)
Routing:
- net +4V: track 40.1 -> 20.7 mm, vias 6 -> 10
- net /EN_PERIPH: track 11.5 -> 29.1 mm, vias 0 -> 3
- net /EXTIO_10: track 0.00 -> 12.7 mm, vias 0 -> 1
- net /EXTIO_9: track 0.00 -> 11.9 mm, vias 0 -> 1
- net /LED_STA: track 0.00 -> 10.2 mm, vias 0 -> 2
- net /EXTIO_8: track 0.00 -> 10.2 mm, vias 0 -> 1
- net /EN_3V3OUT: track 17.1 -> 27.0 mm
- net /ESP_EN: track 21.7 -> 11.9 mm, vias 2 -> 1
- net /EXTIO_7: track 0.00 -> 9.52 mm, vias 0 -> 1
- net /BQ_PGOOD: track 9.20 -> 18.5 mm, vias 2 -> 3
- net /I2S_LRCLK: track 8.61 -> 16.3 mm
- net /BUT2: track 34.1 -> 27.6 mm, vias 3 -> 2
- net +3.3V: track 56.7 -> 62.3 mm, vias 16 -> 17
- net GND: track 87.7 -> 93.1 mm, vias 35 -> 51
- net /LIPO+: track 3.91 -> 7.41 mm
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- added copper zone on In2.Cu, net GND
Other:
- board size 38.8 x 24.5 mm -> 38.7 x 24.5 mm
- board text added: "1"
- board text added: "10"
- board text added: "2"
- board text added: "3"
- board text added: "3v3"
- board text added: "4"
- board text added: "5"
- board text added: "5v"
- board text added: "6"
- board text added: "7"
- board text added: "8"
- board text added: "9"
- board text added: "HBEAT"
- board text added: "Pilkbrain"
- board text added: "d"
- board text added: "dm"
- board text added: "dp"
- board text added: "g"
- board text added: "gnd"
- board text added: "r1 @cb1t"
- board text added: "scl"
- board text added: "sda"
- board text added: "spkr"
- board text removed: "Pilkbrain 10.24 @cb1t"

Commit message: order(?)
Routing:
- net /USBDM: track 29.0 -> 28.2 mm

Commit message: new formfactor placement etc
Parts:
- removed C20: 1u, Capacitor_SMD:C_0402_1005Metric
- removed C24: 10u, Capacitor_SMD:C_0603_1608Metric
- removed C27: 100n, Capacitor_SMD:C_0402_1005Metric
- removed D1, D3: LED_WHITE, LED_SMD:LED_0603_1608Metric
- removed D4: LED_RED, LED_SMD:LED_0603_1608Metric
- removed H1: M2, MountingHole:MountingHole_2.2mm_M2
- removed PAD10: BAT-, Critbit_lib:diy_castellate_2.54
- removed PAD11: EN_3V3, Critbit_lib:diy_castellate_2.54
- removed PAD28: 9, Critbit_lib:diy_castellate_2.54
- removed PAD29: 10, Critbit_lib:diy_castellate_2.54
- removed R12, R31, R32, R33, R34, R6: 10k, Resistor_SMD:R_0402_1005Metric
- removed R35: 100k, Resistor_SMD:R_0402_1005Metric
- added C10: 10u, Capacitor_SMD:C_0603_1608Metric, B.Cu at (117.4, 42.0)
- added CN3: YXT-BB10-24S-02, easyeda2kicad:CONN-SMD_YXT-BB10-24S-02, B.Cu at (110.5, 55.6)
- added U2: XL-1005UWC_C20613596, easyeda2kicad:LED0402-RD_YELLOW, B.Cu at (117.4, 44.9)
- added U5: XL-1005UWC_C20613596, easyeda2kicad:LED0402-RD_YELLOW, B.Cu at (105.4, 53.7)
- added U6: XL-1005UWC_C20613596, easyeda2kicad:LED0402-RD_YELLOW, B.Cu at (107.7, 58.9)
- C14: value 10u -> 1u; footprint Capacitor_SMD:C_0603_1608Metric -> Capacitor_SMD:C_0402_1005Metric
- PAD3, PAD4: value TP -> 10; moved to F.Cu
- R16: value 500k -> 510k/0603; footprint Resistor_SMD:R_0402_1005Metric -> Resistor_SMD:R_0603_1608Metric
- R2: value 10k -> 10k/DNP; footprint Resistor_SMD:R_0402_1005Metric -> Resistor_SMD:R_0603_1608Metric
- R3, R5: value 100k -> 10k
- U1: value TF-123-ARP9H17 -> ~; footprint easyeda2kicad:TF-SMD_TF-123-ARP9H15 -> Critbit_lib:OLED_4Pin_128x64_new
- moved U1 39.8 mm to (71.5, 43.0), turned to 180 degrees
- moved SW2 26.8 mm to (98.8, 56.4), turned to 180 degrees
- moved SW3 25.4 mm to (98.8, 49.0), turned to 180 degrees
- moved C12 24.3 mm to (115.1, 41.1), turned to 0 degrees
- moved PAD19 23.2 mm to (109.8, 38.8), turned to -90 degrees
- moved PAD20 23.2 mm to (112.2, 38.8), turned to -90 degrees
- moved PAD8 23.2 mm to (107.2, 38.8), turned to -90 degrees
- moved PAD9 23.2 mm to (104.8, 38.8), turned to -90 degrees
- moved J1 23.2 mm to (108.8, 67.9), turned to 180 degrees
- moved R37 22.2 mm to (103.0, 67.8), turned to 90 degrees
- moved R1 21.7 mm to (105.5, 40.8)
- moved C14 20.8 mm to (105.8, 42.2), turned to -90 degrees
- moved C19 20.7 mm to (104.3, 44.4), turned to 90 degrees
- moved U3 20.5 mm to (114.6, 43.6), turned to 180 degrees
- moved R24 20.1 mm to (104.7, 46.4), turned to -90 degrees
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Connections:
- R2 pad 1: /SD_DAT1 -> GND
- R2 pad 2: +3.3V -> Net-(U4-TS)
- U1 pad 1: /SD_DAT2 -> unconnected-(U1-GND-Pad1)
- U1 pad 2: /SD_DAT3 -> unconnected-(U1-VCC-Pad2)
- U1 pad 3: /SD_CMD -> unconnected-(U1-SCL-Pad3)
- U1 pad 4: +3.3V -> unconnected-(U1-SDA-Pad4)
- U13 pad 11: unconnected-(U13-GPIO6/ADC1_CH5-Pad11) -> /EXTIO_1
- U13 pad 12: unconnected-(U13-GPIO7/ADC1_CH6-Pad12) -> /EN_3V3OUT
- U13 pad 13: /BUT2 -> /LED_STA
- U13 pad 14: /EXTIO_1 -> /EXTIO_8
- U13 pad 15: /VBAT_MEAS -> /EXTIO_7
- U13 pad 16: /I2S_LRCLK -> /EXTIO_6
- U13 pad 17: /I2S_DAT -> /EXTIO_5
- U13 pad 18: /I2S_CLK -> /EXTIO_4
- U13 pad 19: /EN_3V3OUT -> /EXTIO_3
- U13 pad 24: /SD_DAT3 -> /VBAT_MEAS
- U13 pad 27: /SD_CMD -> /WS2812_OUT
- U13 pad 36: /SD_DAT2 -> /SD_DAT3
- U13 pad 37: /WS2812_OUT -> /SD_DAT2
- U13 pad 38: unconnected-(U13-GPIO33-Pad38) -> /SD_CLK
- U13 pad 39: /SD_CLK -> /SD_CMD
- U13 pad 40: /I2C_SCL -> /SD_DAT0
- U13 pad 41: /SD_DAT0 -> /SD_DAT1
- U13 pad 42: /I2C_SDA -> /SD_DET
- U13 pad 43: /SD_DAT1 -> /BQ_PGOOD
- U13 pad 44: /EXTIO_10 -> /BQ_CHG
- U13 pad 45: /EXTIO_8 -> /I2S_CLK
- U13 pad 47: /EXTIO_7 -> /I2S_DAT
- U13 pad 48: /EXTIO_9 -> /BUT2
- U13 pad 51: /BQ_PGOOD -> /I2S_LRCLK
- U13 pad 52: /LED_STA -> unconnected-(U13-GPIO46-Pad52)
- U13 pad 6: /EXTIO_6 -> unconnected-(U13-GPIO1/ADC1_CH0-Pad6)
- U13 pad 7: /EXTIO_5 -> unconnected-(U13-GPIO2/ADC1_CH1-Pad7)
- U13 pad 8: /EXTIO_4 -> unconnected-(U13-GPIO3/ADC1_CH2-Pad8)
- U13 pad 9: /EXTIO_3 -> unconnected-(U13-GPIO4/ADC1_CH3-Pad9)
Routing:
- net GND: track 93.1 -> 41.2 mm, vias 51 -> 6
- net +3.3V: track 62.3 -> 19.0 mm, vias 17 -> 1
- net /BOOT_BUT1: track 44.4 -> 14.4 mm, vias 4 -> 1
- net /USBDP: track 30.8 -> 9.23 mm, vias 2 -> 1
- net /I2C_SDA: track 21.4 -> 0.71 mm, vias 3 -> 1
- net /EN_PERIPH: track 29.1 -> 9.56 mm, vias 3 -> 2
- net /WS2812_OUT: track 20.8 -> 1.93 mm, vias 2 -> 1
- net /I2C_SCL: track 18.5 -> 0.82 mm, vias 2 -> 1
- net Net-(U4-TS): track 15.1 -> 0.00 mm, vias 1 -> 0
- net /EN_3V3OUT: track 27.0 -> 12.2 mm
- net /I2S_LRCLK: track 16.3 -> 1.85 mm
- net /USBDM: track 28.2 -> 14.3 mm
- net /BUT2: track 27.6 -> 13.9 mm
- net /EXTIO_10: track 12.9 -> 0.00 mm, vias 1 -> 0
- net /EXTIO_9: track 11.9 -> 0.00 mm, vias 1 -> 0
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- added copper zone on F.Cu, net VBUS
- removed copper zone on In2.Cu, net +3.3V
- removed copper zone on B.Cu, net +4V
- removed copper zone on F.Cu, net +4V
- removed copper zone on In2.Cu, net /3V3_OUT
- removed copper zone on In2.Cu, net /LIPO+
- removed copper zone on In2.Cu, net /WS2812_VDD
- removed copper zone on In2.Cu, net GND
Other:
- board size 38.7 x 24.5 mm -> 24.3 x 32.1 mm
- board text added: "@cb1t"
- board text added: "STA"
- board text added: "rev2"
- board text removed: "HBEAT"
- board text removed: "r1 @cb1t"
