File: pilkbrain.kicad_pcb (KiCad board)
At the start: 4 copper layers, 24.3 x 32.1 mm, 94 parts, among them CN3 YXT-BB10-24S-02, J1 USB_C_Receptacle_USB2.0, J2 Conn_01x05, SW2 EVQPUC02K, SW3 EVQPUC02K, U13 ESP32-S3, U2 XL-1005UWC_C20613596, U3 SPX3819M5-L-3-3, U4 BQ24073RGT, U5 XL-1005UWC_C20613596, U6 XL-1005UWC_C20613596, U7 MT9700, U8 MAX98357AEWL+T, U9 MT9700, Y1 XO-40M, Y2 XO-32K

Commit message: rev2 prod?
Parts:
- removed J1: USB_C_Receptacle_USB2.0, Connector_USB:USB_C_Receptacle_HRO_TYPE-C-31-M-12
- removed R36, R37: 5.1k, Resistor_SMD:R_0402_1005Metric
- removed U1: ~, Critbit_lib:OLED_4Pin_128x64_new
- added R12: 5.1k, Resistor_SMD:R_0402_1005Metric, B.Cu at (108.5, 67.8)
- added R6: 5.1k, Resistor_SMD:R_0402_1005Metric, B.Cu at (108.5, 63.2)
- added USB1: GT-USB-7055E, easyeda2kicad:USB-C-SMD_GT-USB-7055E, B.Cu at (108.5, 65.4)
- moved R11 0.54 mm to (117.6, 54.3), turned to -90 degrees
- moved C29 0.51 mm to (116.0, 53.8)
- moved R10 0.46 mm to (116.0, 54.8)
- moved R4 0.25 mm to (108.5, 40.6)
- moved AE1 0.20 mm to (99.3, 40.0)
- moved PAD15 0.20 mm to (115.5, 38.9)
- moved PAD18 0.20 mm to (117.5, 38.9)
- moved PAD14 0.15 mm to (120.0, 50.8)
- moved PAD16 0.15 mm to (120.1, 42.6)
- moved PAD17 0.15 mm to (120.0, 53.0)
- moved PAD24 0.15 mm to (120.1, 48.6)
- moved PAD25 0.15 mm to (120.1, 46.6)
- moved PAD26 0.15 mm to (120.1, 44.6)
- moved PAD3 0.15 mm to (120.1, 55.2)
- moved PAD4 0.15 mm to (120.1, 57.4)
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Connections:
- CN3 pad 15: unconnected-(CN3-Pad15) -> +3.3V
- CN3 pad 16: unconnected-(CN3-Pad16) -> +3.3V
- CN3 pad 18: /I2C_SDA -> /I2C_SCL
- CN3 pad 19: /I2C_SCL -> /I2C_SDA
- CN3 pad 20: /3V3_OUT -> VBUS
- CN3 pad 21: /3V3_OUT -> VBUS
- PAD3 pad 1: Net-(U8-OUTN) -> Net-(U8-OUTP)
- PAD4 pad 1: Net-(U8-OUTP) -> Net-(U8-OUTN)
- U13 pad 16: /EXTIO_6 -> /EN_PERIPH
- U13 pad 23: /EN_PERIPH -> /I2S_DAT
- U13 pad 27: /WS2812_OUT -> /SD_DAT2
- U13 pad 37: /SD_DAT2 -> /I2S_CLK
- U13 pad 42: /SD_DET -> unconnected-(U13-GPIO37-Pad42)
- U13 pad 45: /I2S_CLK -> /I2C_SCL
- U13 pad 47: /I2S_DAT -> /I2C_SDA
- U13 pad 7: unconnected-(U13-GPIO2/ADC1_CH1-Pad7) -> /EXTIO_6
- U13 pad 8: unconnected-(U13-GPIO3/ADC1_CH2-Pad8) -> /SD_DET
- U13 pad 9: unconnected-(U13-GPIO4/ADC1_CH3-Pad9) -> /WS2812_OUT
Routing:
- net GND: track 41.2 -> 110.1 mm, vias 6 -> 45
- net /I2C_SDA: track 0.71 -> 23.4 mm, vias 1 -> 2
- net /I2C_SCL: track 0.82 -> 22.8 mm, vias 1 -> 2
- net VBUS: track 5.48 -> 27.1 mm, vias 2 -> 4
- net +3.3V: track 19.0 -> 36.0 mm, vias 1 -> 14
- net +4V: track 10.6 -> 27.3 mm, vias 2 -> 6
- net /WS2812_OUT: track 1.93 -> 17.5 mm
- net /I2S_CLK: track 1.59 -> 12.7 mm
- net /I2S_DAT: track 1.55 -> 12.0 mm
- net /I2S_LRCLK: track 1.85 -> 12.0 mm
- net /USBDP: track 9.23 -> 18.5 mm, vias 1 -> 3
- net /USBDM: track 14.3 -> 23.3 mm, vias 1 -> 4
- net /BQ_PGOOD: track 9.74 -> 18.6 mm, vias 1 -> 3
- net /BOOT_BUT1: track 14.4 -> 21.1 mm, vias 1 -> 2
- net /SD_DET: track 8.07 -> 13.9 mm
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- added copper zone on In1.Cu, net +3.3V
- added copper zone on In1.Cu, net +4V
- added copper zone on In2.Cu, net GND
- removed copper zone on In1.Cu, net GND
Other:
- board size 24.3 x 32.1 mm -> 24.3 x 30.5 mm
- board text added: "S+"
- board text added: "S-"
- board text added: "rev2 @cb1t"
- board text removed: "-"
- board text removed: "10"
- board text removed: "9"
- board text removed: "<-insert bepis"
- board text removed: "@cb1t"
- board text removed: "Made at Hackerspace Pomerania hsp.sh"
- board text removed: "dm"
- board text removed: "dp"
- board text removed: "github.com/ hspsh/pilkbadge"
- board text removed: "gnd"
- board text removed: "insert milk->"
- board text removed: "rev2"
- board text removed: "spkr"

Commit message: 3rd redo but good this time
Parts:
- removed C26: 1u, Capacitor_SMD:C_0402_1005Metric
- removed C32: 10u, Capacitor_SMD:C_0603_1608Metric
- removed CN3: YXT-BB10-24S-02, easyeda2kicad:CONN-SMD_YXT-BB10-24S-02
- removed J2: Conn_01x05, Connector_PinHeader_1.27mm:PinHeader_1x05_P1.27mm_Vertical
- removed PAD22: WS2812_OUT, Critbit_lib:diy_castellate_2.54
- removed PAD23: GND, Critbit_lib:diy_castellate_2.54
- removed SW2: EVQPUC02K, easyeda2kicad:SW-SMD_EVQPUD02K
- removed USB1: GT-USB-7055E, easyeda2kicad:USB-C-SMD_GT-USB-7055E
- added C20: 100n, Capacitor_SMD:C_0402_1005Metric, B.Cu at (114.8, 52.0)
- added C22: 10u, Capacitor_SMD:C_0402_1005Metric, B.Cu at (103.8, 42.4)
- added C24: 100n, Capacitor_SMD:C_0402_1005Metric, B.Cu at (106.4, 55.8)
- added CN1: SM02B-SRSS-TB (LF)(SN), easyeda2kicad:CONN-SMD_2P-P1.00_SM02B-SRSS-TB-LF-SN, B.Cu at (114.5, 43.4)
- added PAD10: PAD_T, Critbit_lib:diy_castellate_tight, B.Cu at (118.7, 42.9)
- added PAD11: PAD_T, Critbit_lib:diy_castellate_tight, B.Cu at (118.7, 41.1)
- added PAD28: PAD_T, Critbit_lib:diy_castellate_tight, B.Cu at (116.2, 65.0)
- added R20: 10k, Resistor_SMD:R_0402_1005Metric, B.Cu at (105.2, 54.4)
- added R21: 10k, Resistor_SMD:R_0402_1005Metric, B.Cu at (106.2, 54.4)
- added R22: 10k, Resistor_SMD:R_0402_1005Metric, B.Cu at (108.0, 55.4)
- added R23: 10k, Resistor_SMD:R_0402_1005Metric, B.Cu at (108.6, 53.9)
- added R25: 10k, Resistor_SMD:R_0402_1005Metric, B.Cu at (110.5, 55.8)
- added R26: 100k, Resistor_SMD:R_0402_1005Metric, B.Cu at (102.0, 56.9)
- added SW1: TS24CA, easyeda2kicad:SW-SMD_TS24CA, B.Cu at (99.2, 48.6)
- added U1: TYPE-C 16P LTH8.8, easyeda2kicad:USB-C-SMD_TYPE-C-16P-LTH8.8, B.Cu at (108.2, 68.5)
- added U10: A-SP1102AR6GHC-A01-2C, easyeda2kicad:LED-SMD_4P-L3.0-W1.5_A-SP1102AR6GHC-A01-2C, B.Cu at (98.7, 53.4)
- added U11: TF-123-ARP9H17, easyeda2kicad:TF-SMD_TF-123-ARP9H15, B.Cu at (107.2, 59.9)
- added U12: SM03B-SRSS-TB(LF)(SN)(P), easyeda2kicad:CONN-SMD_SM03B-SRSS-TB-LF-SN-P, B.Cu at (116.6, 62.2)
- C10, C12, C15: value 10u -> 1u; footprint Capacitor_SMD:C_0603_1608Metric -> Capacitor_SMD:C_0402_1005Metric
- C11: value 10u -> 47uF/0805; footprint Capacitor_SMD:C_0603_1608Metric -> Capacitor_SMD:C_0805_2012Metric
- C13, C16, C9: footprint Capacitor_SMD:C_0603_1608Metric -> Capacitor_SMD:C_0402_1005Metric
- PAD1: value BAT- -> PAD_T; footprint Critbit_lib:diy_castellate_2.54 -> Critbit_lib:diy_castellate_tight
- PAD12: value 5V -> PAD_T; footprint Critbit_lib:diy_castellate_2.54 -> Critbit_lib:diy_castellate_tight
- PAD13: value GND -> PAD_T; footprint Critbit_lib:diy_castellate_2.54 -> Critbit_lib:diy_castellate_tight
- PAD14: value 3 -> PAD_T; footprint Critbit_lib:diy_castellate_2.54 -> Critbit_lib:diy_castellate_tight; moved to B.Cu
- PAD15: value 2 -> PAD_T; footprint Critbit_lib:diy_castellate_2.54 -> Critbit_lib:diy_castellate_tight; moved to B.Cu
- PAD16: value 7 -> PAD_T; footprint Critbit_lib:diy_castellate_2.54 -> Critbit_lib:diy_castellate_tight
- PAD17: value GND -> PAD_T; footprint Critbit_lib:diy_castellate_2.54 -> Critbit_lib:diy_castellate_tight; moved to B.Cu
- PAD18: value 1 -> PAD_T; footprint Critbit_lib:diy_castellate_2.54 -> Critbit_lib:diy_castellate_tight; moved to B.Cu
- PAD19: value 3V3_OUT -> PAD; moved to B.Cu
- PAD2: value BAT+ -> PAD_T; footprint Critbit_lib:diy_castellate_2.54 -> Critbit_lib:diy_castellate_tight
- PAD20: value GND -> PAD; moved to B.Cu
- PAD21: value 4V_OUT -> PAD
- PAD24: value 4 -> PAD_T; footprint Critbit_lib:diy_castellate_2.54 -> Critbit_lib:diy_castellate_tight; moved to B.Cu
- PAD25: value 5 -> PAD_T; footprint Critbit_lib:diy_castellate_2.54 -> Critbit_lib:diy_castellate_tight; moved to B.Cu
- PAD26: value 6 -> PAD_T; footprint Critbit_lib:diy_castellate_2.54 -> Critbit_lib:diy_castellate_tight; moved to B.Cu
- PAD27: value 8 -> PAD_T; footprint Critbit_lib:diy_castellate_2.54 -> Critbit_lib:diy_castellate_tight
- PAD3, PAD4: value 10 -> PAD_T; footprint Critbit_lib:diy_castellate_2.54 -> Critbit_lib:diy_castellate_tight; moved to B.Cu
- PAD5: value TC -> PAD_T; footprint Critbit_lib:diy_castellate_2.54 -> Critbit_lib:diy_castellate_tight
- PAD6: value DM -> PAD_T; footprint Critbit_lib:diy_castellate_2.54 -> Critbit_lib:diy_castellate_tight
- PAD7: value DP -> PAD_T; footprint Critbit_lib:diy_castellate_2.54 -> Critbit_lib:diy_castellate_tight
- PAD8: value SCL -> PAD; moved to B.Cu
- PAD9: value SDA -> PAD; moved to B.Cu
- R10: value 10k -> 100k
- SW3: value EVQPUC02K -> TS24CA; footprint easyeda2kicad:SW-SMD_EVQPUD02K -> easyeda2kicad:SW-SMD_TS24CA
- U13: footprint Package_DFN_QFN:QFN-56-1EP_7x7mm_P0.4mm_EP4x4mm -> Package_DFN_QFN:QFN-56-1EP_7x7mm_P0.4mm_EP5.6x5.6mm
- U3: value SPX3819M5-L-3-3 -> SSP7615-33DFR; footprint Package_TO_SOT_SMD:SOT-23-5 -> easyeda2kicad:DFN-4_L1.0-W1.0-P0.65-BL-EP
- U7: value MT9700 -> AP2552FDC-7; footprint easyeda2kicad:SOT-23-5_L3.0-W1.7-P0.95-LS2.8-BR -> easyeda2kicad:WDFN-6_L2.0-W2.0-P0.65-BL-EP-1
- U9: value MT9700 -> SSP7615-33DFR; footprint easyeda2kicad:SOT-23-5_L3.0-W1.7-P0.95-LS2.8-BR -> easyeda2kicad:DFN-4_L1.0-W1.0-P0.65-BL-EP
- Y1: footprint Crystal:Crystal_SMD_3225-4Pin_3.2x2.5mm -> Crystal:Crystal_SMD_2520-4Pin_2.5x2.0mm
- Y2: footprint Crystal:Crystal_SMD_3215-2Pin_3.2x1.5mm -> Crystal:Crystal_SMD_2012-2Pin_2.0x1.2mm
- moved PAD17 33.2 mm to (89.8, 66.8), turned to 90 degrees
- moved U2 26.4 mm to (92.5, 53.6)
- moved R15 24.4 mm to (92.2, 51.2)
- moved PAD4 22.7 mm to (98.7, 64.9), turned to 90 degrees
- moved PAD21 22.4 mm to (114.5, 39.5), turned to -90 degrees
- moved PAD3 22.0 mm to (100.4, 65.0), turned to 90 degrees
- moved C10 20.6 mm to (102.1, 55.8), turned to 0 degrees
- moved R2 18.2 mm to (116.5, 55.9), turned to -90 degrees
- moved R8 18.2 mm to (90.6, 51.4)
- moved C12 18.0 mm to (101.8, 53.2)
- moved PAD18 18.0 mm to (118.7, 56.9), turned to 180 degrees
- moved U6 17.9 mm to (90.5, 53.3)
- moved PAD1 16.7 mm to (114.5, 65.0)
- moved PAD15 16.5 mm to (118.7, 55.1), turned to 180 degrees
- moved R16 15.4 mm to (110.7, 43.5), turned to -90 degrees
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Connections:
- C11 pad 1: +4V -> /LIPO+
- C13 pad 1: /LIPO+ -> +4V
- C14 pad 1: +3.3V -> +4V
- PAD1 pad 1: GND -> /EXTIO_12
- PAD17 pad 1: GND -> /EXTIO_17
- PAD2 pad 1: /LIPO+ -> /EXTIO_13
- PAD3 pad 1: Net-(U8-OUTP) -> /EXTIO_14
- PAD4 pad 1: Net-(U8-OUTN) -> /EXTIO_15
- PAD5 pad 1: Net-(U4-TS) -> /EXTIO_16
- R10 pad 2: Net-(U7-SET) -> Net-(U7-ILIM)
- R17 pad 1: GND -> /SD_DAT1
- R17 pad 2: Net-(U9-SET) -> +3.3V
- SW3 pad 2: /BOOT_BUT1 -> (no net)
- SW3 pad 4: /BOOT_BUT1 -> /BUT2
- U13 pad 27: /SD_DAT2 -> unconnected-(U13-GPIO21-Pad27)
- U13 pad 36: /SD_DAT3 -> /SD_DAT2
- U13 pad 37: /I2S_CLK -> /SD_DAT3
- U13 pad 38: /SD_CLK -> /SD_CMD
- U13 pad 39: /SD_CMD -> /SD_DET
- U13 pad 40: /SD_DAT0 -> /SD_CLK
- U13 pad 41: /SD_DAT1 -> /SD_DAT0
- U13 pad 42: unconnected-(U13-GPIO37-Pad42) -> /SD_DAT1
- U13 pad 8: /SD_DET -> unconnected-(U13-GPIO3/ADC1_CH2-Pad8)
- U3 pad 1: +4V -> /3V3_OUT
- U3 pad 3: +4V -> /EN_3V3OUT
- U3 pad 4: unconnected-(U3-BP-Pad4) -> +4V
- U3 pad 5: +3.3V -> unconnected-(U3-EP-Pad5)
- U7 pad 2: GND -> Net-(U7-ILIM)
- U7 pad 3: Net-(U7-SET) -> unconnected-(U7-~{FAULT}-Pad3)
- U7 pad 5: +4V -> GND
- U9 pad 1: /3V3_OUT -> +3.3V
- U9 pad 3: Net-(U9-SET) -> +4V
- U9 pad 4: /EN_3V3OUT -> +4V
- U9 pad 5: +3.3V -> unconnected-(U9-EP-Pad5)
Routing:
- net GND: track 110.1 -> 0.00 mm, vias 45 -> 0
- net +3.3V: track 36.0 -> 1.01 mm, vias 14 -> 0
- net +4V: track 27.3 -> 0.00 mm, vias 6 -> 0
- net VBUS: track 27.1 -> 0.00 mm, vias 4 -> 0
- net /WS2812_VDD: track 25.1 -> 1.28 mm, vias 3 -> 0
- net /USBDM: track 23.3 -> 0.00 mm, vias 4 -> 0
- net /I2C_SDA: track 23.4 -> 1.08 mm, vias 2 -> 0
- net /BOOT_BUT1: track 21.1 -> 0.00 mm, vias 2 -> 0
- net /I2C_SCL: track 22.8 -> 3.63 mm, vias 2 -> 0
- net /BUT2: track 19.2 -> 0.00 mm, vias 2 -> 0
- net /BQ_PGOOD: track 18.6 -> 0.00 mm, vias 3 -> 0
- net /USBDP: track 18.5 -> 0.00 mm, vias 3 -> 0
- net /WS2812_OUT: track 17.5 -> 0.00 mm, vias 1 -> 0
- net /ESP_EN: track 15.4 -> 0.00 mm, vias 2 -> 0
- net /EN_PERIPH: track 13.5 -> 0.00 mm, vias 2 -> 0
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Other:
- board size 24.3 x 30.5 mm -> 21.9 x 33 mm
