File: pilkbrain.kicad_pcb (KiCad board)
At the start: 4 copper layers, 21.9 x 33 mm, 103 parts, among them CN1 SM02B-SRSS-TB (LF)(SN), SW1 TS24CA, SW3 TS24CA, U1 TYPE-C 16P LTH8.8, U10 A-SP1102AR6GHC-A01-2C, U11 TF-123-ARP9H17, U12 SM03B-SRSS-TB(LF)(SN)(P), U13 ESP32-S3, U2 XL-1005UWC_C20613596, U3 SSP7615-33DFR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

Commit message: before order
Parts:
- removed PAD17, PAD5: PAD_T, Critbit_lib:diy_castellate_tight
- removed U10: A-SP1102AR6GHC-A01-2C, easyeda2kicad:LED-SMD_4P-L3.0-W1.5_A-SP1102AR6GHC-A01-2C
- added R27: 47k, Resistor_SMD:R_0402_1005Metric, B.Cu at (110.7, 42.0)
- added TP1: TP, TestPoint:TestPoint_Pad_D1.0mm, F.Cu at (109.1, 47.0)
- added TP10: TP, TestPoint:TestPoint_Pad_D1.0mm, F.Cu at (114.2, 45.9)
- added TP11: TP, TestPoint:TestPoint_Pad_D1.0mm, F.Cu at (112.7, 44.5)
- added TP7: TP, TestPoint:TestPoint_Pad_D1.0mm, F.Cu at (107.8, 43.7)
- added TP9: TP, TestPoint:TestPoint_Pad_D1.0mm, F.Cu at (114.2, 43.1)
- C3: value 1u -> 10u
- R10, R26: value 100k -> 47k
- R16: value 510k/0603 -> 510k
- moved R13 18.2 mm to (117.4, 53.5), turned to -90 degrees
- moved R9 11.1 mm to (104.3, 53.8), turned to 180 degrees
- moved R8 9.97 mm to (99.5, 55.8), turned to 180 degrees
- moved R3 8.74 mm to (111.7, 42.0), turned to 90 degrees
- moved R5 8.37 mm to (111.2, 43.5)
- moved U6 8.27 mm to (98.0, 56.9), turned to -90 degrees
- moved R15 7.56 mm to (99.5, 53.2), turned to 180 degrees
- moved R24 6.72 mm to (102.6, 45.6), turned to 0 degrees
- moved R10 5.87 mm to (117.5, 51.5), turned to 90 degrees
- moved U2 5.76 mm to (98.0, 52.0)
- moved C17 5.32 mm to (111.5, 44.6)
- moved C18 4.56 mm to (100.2, 61.0), turned to 90 degrees
- moved U5 4.47 mm to (98.0, 54.5)
- moved C19 4.27 mm to (101.1, 46.1), turned to -90 degrees
- moved R6 4.20 mm to (108.3, 66.5)
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Connections:
- CN1 pad 1: Net-(U8-OUTN) -> Net-(U8-OUTP)
- CN1 pad 2: Net-(U8-OUTP) -> Net-(U8-OUTN)
- CN1 pad 3: unconnected-(CN1-Pad3) -> GND
- CN1 pad 4: unconnected-(CN1-Pad4) -> GND
- PAD1 pad 1: /EXTIO_12 -> /BQ_PGOOD
- PAD2 pad 1: /EXTIO_13 -> /BOOT_BUT1
- PAD28 pad 1: /EXTIO_11 -> /BQ_CHG
- PAD3 pad 1: /EXTIO_14 -> /TARG_TX
- PAD4 pad 1: /EXTIO_15 -> /TARG_RX
- SW1 pad 2: (no net) -> GND
- SW3 pad 2: (no net) -> GND
- U13 pad 10: /EXTIO_2 -> /EXTIO_8
- U13 pad 11: /EXTIO_1 -> /EXTIO_9
- U13 pad 12: /EN_3V3OUT -> /I2S_CLK
- U13 pad 13: /LED_STA -> /VBAT_MEAS
- U13 pad 14: /EXTIO_8 -> /I2S_DAT
- U13 pad 15: /EXTIO_7 -> /PERIPH_FAULT
- U13 pad 16: /EN_PERIPH -> /I2S_LRCLK
- U13 pad 17: /EXTIO_5 -> /EXTIO_7
- U13 pad 18: /EXTIO_4 -> /EXTIO_6
- U13 pad 19: /EXTIO_3 -> /EXTIO_5
- U13 pad 23: /I2S_DAT -> /EN_PERIPH
- U13 pad 24: /VBAT_MEAS -> /EXTIO_3
- U13 pad 27: unconnected-(U13-GPIO21-Pad27) -> /EXTIO_1
- U13 pad 45: /I2C_SCL -> /LED_STA
- U13 pad 47: /I2C_SDA -> /EXTIO_2
- U13 pad 51: /I2S_LRCLK -> /EXTIO_4
- U13 pad 52: unconnected-(U13-GPIO46-Pad52) -> /3V3_MEAS
- U13 pad 6: unconnected-(U13-GPIO1/ADC1_CH0-Pad6) -> /I2C_SDA
- U13 pad 7: /EXTIO_6 -> /I2C_SCL
- U13 pad 8: unconnected-(U13-GPIO3/ADC1_CH2-Pad8) -> /EN_3V3OUT
- U13 pad 9: /WS2812_OUT -> /EXTIO_10
- U3 pad 5: unconnected-(U3-EP-Pad5) -> GND
- U7 pad 3: unconnected-(U7-~{FAULT}-Pad3) -> /PERIPH_FAULT
- U9 pad 5: unconnected-(U9-EP-Pad5) -> GND
Routing:
- net GND: track 0.00 -> 106.6 mm, vias 0 -> 72
- net +3.3V: track 1.01 -> 64.9 mm, vias 0 -> 16
- net +4V: track 0.00 -> 42.7 mm, vias 0 -> 9
- net /BQ_PGOOD: track 0.00 -> 31.0 mm, vias 0 -> 3
- net /BOOT_BUT1: track 0.00 -> 30.7 mm, vias 0 -> 4
- net VBUS: track 0.00 -> 30.1 mm, vias 0 -> 7
- net /BQ_CHG: track 0.00 -> 25.8 mm, vias 0 -> 2
- net /USBDM: track 0.00 -> 24.5 mm, vias 0 -> 3
- net /TARG_TX: track 0.00 -> 22.6 mm, vias 0 -> 1
- net /TARG_RX: track 0.00 -> 22.4 mm, vias 0 -> 1
- net /WS2812_VDD: track 1.28 -> 22.2 mm, vias 0 -> 5
- net /USBDP: track 0.00 -> 20.9 mm, vias 0 -> 1
- net /BUT2: track 0.00 -> 20.0 mm, vias 0 -> 2
- net /EXTIO_4: track 0.00 -> 18.6 mm, vias 0 -> 1
- net /EXTIO_2: track 0.00 -> 17.4 mm, vias 0 -> 1
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- added copper zone on F.Cu, net +4V
- added copper zone on In1.Cu, net /WS2812_VDD
- added copper zone on In1.Cu, net GND
Other:
- board size 21.9 x 33 mm -> 22.9 x 33 mm
- board text added: "-"
- board text added: "1 0"
- board text added: "46"
- board text added: "4v"
- board text added: "9"
- board text added: "T"
- board text added: "b1"
- board text added: "b2"
- board text added: "boot"
- board text added: "clk"
- board text added: "dat"
- board text added: "en"
- board text added: "gnd"
- board text added: "lrc"
- board text added: "rev3 @cb1t"
- board text added: "rx"
- board text added: "tx"
- board text removed: "5v"
- board text removed: "Tc"
- board text removed: "d"
- board text removed: "g"
- board text removed: "rev2 @cb1t"

Commit message: wrong holes
Parts:
- moved PAD10 0.25 mm to (119.2, 43.1)
- moved PAD11 0.25 mm to (119.2, 41.4)
- moved PAD14 0.25 mm to (119.2, 53.6)
- moved PAD15 0.25 mm to (119.2, 55.4)
- moved PAD16 0.25 mm to (119.2, 46.6)
- moved PAD18 0.25 mm to (119.2, 57.1)
- moved PAD24 0.25 mm to (119.2, 51.9)
- moved PAD25 0.25 mm to (119.2, 50.1)
- moved PAD26 0.25 mm to (119.2, 48.4)
- moved PAD27 0.25 mm to (119.2, 44.9)
- moved U12 0.21 mm to (116.1, 62.1)
Routing:
- net /EXTIO_9: track 13.4 -> 14.7 mm
- net /EXTIO_2: track 17.4 -> 16.5 mm
- net /EXTIO_1: track 10.4 -> 9.50 mm
- net /EXTIO_5: track 8.35 -> 7.68 mm
- net GND: track 106.6 -> 106.7 mm, vias 72 -> 71
Other:
- board size 22.9 x 33 mm -> 22 x 33 mm
- board text added: "g"

Commit message: another element swappage
Parts:
- moved C3 0.30 mm to (101.5, 53.0)
- moved C7 0.30 mm to (100.7, 47.6)
- moved C8 0.30 mm to (101.5, 52.0)
- moved L3 0.22 mm to (102.6, 47.6)
- moved C17 0.20 mm to (111.6, 44.4)
- moved Y2 0.18 mm to (113.5, 48.8)
- moved C21 0.16 mm to (108.5, 44.4)
- moved R5 0.11 mm to (111.2, 43.4)
- moved R7 0.11 mm to (107.0, 43.8)
- moved C14 0.11 mm to (107.2, 41.9)
- moved U3 0.10 mm to (108.5, 41.9)
- moved R18 0.10 mm to (108.6, 43.4)
- moved C15 0.10 mm to (109.8, 41.9)
- moved R3 0.09 mm to (111.7, 42.0)
- moved R27 0.08 mm to (110.8, 42.0)
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Connections:
- U13 pad 10: /EXTIO_8 -> /EXTIO_9
- U13 pad 11: /EXTIO_9 -> /I2S_CLK
- U13 pad 12: /I2S_CLK -> /EXTIO_8
Routing:
- net /BQ_CHG: track 25.8 -> 41.2 mm, vias 2 -> 3
- net /WS2812_VDD: track 22.2 -> 31.6 mm
- net GND: track 106.7 -> 100.0 mm, vias 71 -> 70
- net +3.3V: track 64.9 -> 58.4 mm
- net +4V: track 42.7 -> 36.3 mm
- net VBUS: track 30.1 -> 25.8 mm
- net /BQ_PGOOD: track 31.0 -> 34.7 mm
- net /PERIPH_FAULT: track 11.5 -> 13.7 mm
- net /EXTIO_9: track 14.7 -> 13.5 mm
- net Net-(U13-XTAL_N): track 7.25 -> 6.25 mm
- net /EXTIO_8: track 12.4 -> 11.6 mm
- net /3V3_MEAS: track 11.0 -> 11.6 mm
- net /BUT2: track 20.0 -> 20.5 mm

Commit message: finish route?
Parts:
- removed C18: 100n, Capacitor_SMD:C_0402_1005Metric
- removed R19: 10k, Resistor_SMD:R_0402_1005Metric
- removed SW3: TS24CA, easyeda2kicad:SW-SMD_TS24CA
- added PAD17: PAD_T, Critbit_lib:diy_castellate_tight, B.Cu at (119.2, 62.5)
- added PAD23: PAD_T, Critbit_lib:diy_castellate_tight, B.Cu at (116.8, 39.5)
- added PAD5: PAD_T, Critbit_lib:diy_castellate_tight, B.Cu at (117.2, 64.5)
- moved PAD4 21.5 mm to (119.2, 60.8), turned to 180 degrees
- moved PAD3 20.0 mm to (119.2, 59.0), turned to 180 degrees
- moved PAD1 15.3 mm to (99.2, 64.5)
- moved PAD28 15.0 mm to (101.2, 64.5)
- moved PAD2 13.1 mm to (115.2, 64.5)
- moved R9 10.1 mm to (100.2, 63.0)
- moved R24 9.57 mm to (98.4, 54.2), turned to 180 degrees
- moved R15 8.20 mm to (99.3, 45.0), turned to -90 degrees
- moved R8 7.41 mm to (98.3, 63.0)
- moved R2 7.09 mm to (111.4, 60.4), turned to 90 degrees
- moved R26 6.80 mm to (102.1, 63.0), turned to 180 degrees
- moved U2 6.55 mm to (98.0, 45.5)
- moved C10 3.78 mm to (100.7, 52.5), turned to 90 degrees
- moved U6 3.36 mm to (98.0, 60.2)
- moved R17 3.32 mm to (100.7, 54.2), turned to 180 degrees
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Connections:
- PAD2 pad 1: /BOOT_BUT1 -> /EXTIO_0
- R3 pad 2: /WS2812_VDD -> Net-(PAD23-Pad1)
- U13 pad 15: /PERIPH_FAULT -> /EXTIO_7
- U13 pad 17: /EXTIO_7 -> /EN_PERIPH
- U13 pad 23: /EN_PERIPH -> /EXTIO_3
- U13 pad 24: /EXTIO_3 -> /BQ_CHG
- U13 pad 27: /EXTIO_1 -> /BQ_PGOOD
- U13 pad 38: /SD_CMD -> /EXTIO_1
- U13 pad 39: /SD_DET -> /EXTIO_2
- U13 pad 40: /SD_CLK -> /SD_CMD
- U13 pad 41: /SD_DAT0 -> /SD_CLK
- U13 pad 42: /SD_DAT1 -> /SD_DAT0
- U13 pad 43: /BQ_PGOOD -> /SD_DAT1
- U13 pad 44: /BQ_CHG -> /SD_DET
- U13 pad 45: /LED_STA -> /EXTIO_0
- U13 pad 47: /EXTIO_2 -> /PERIPH_FAULT
- U13 pad 48: /BUT2 -> /LED_STA
Routing:
- net /EXTIO_0: track 0.00 -> 31.2 mm, vias 0 -> 3
- net /BUT2: track 20.5 -> 0.00 mm, vias 2 -> 0
- net /TARG_RX: track 22.5 -> 36.3 mm, vias 1 -> 3
- net /TARG_TX: track 22.2 -> 35.4 mm, vias 1 -> 3
- net /BQ_CHG: track 41.2 -> 28.0 mm, vias 3 -> 1
- net +4V: track 36.3 -> 24.0 mm, vias 9 -> 10
- net /BOOT_BUT1: track 31.1 -> 42.9 mm
- net /WS2812_VDD: track 31.6 -> 21.9 mm
- net /BQ_PGOOD: track 34.7 -> 25.5 mm, vias 3 -> 1
- net /LIPO+: track 10.1 -> 2.41 mm
- net VBUS: track 25.8 -> 18.7 mm, vias 7 -> 6
- net /EXTIO_1: track 9.57 -> 15.6 mm
- net Net-(PAD23-Pad1): track 0.00 -> 5.32 mm
- net GND: track 100.0 -> 104.7 mm, vias 70 -> 63
- net /LED_STA: track 7.28 -> 11.0 mm, vias 2 -> 3
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- added copper zone on B.Cu, net /LIPO+
- added copper zone on In1.Cu, net VBUS
- removed copper zone on In1.Cu, net GND
Other:
- board size 22 x 33 mm -> 22 x 30.5 mm
- board text added: "@cb1t"
- board text added: "rev3"
- board text removed: "rev3 @cb1t"

Commit message: little schematic cleanup, add PDF and render image
Parts:
- moved C22 0.50 mm to (103.7, 41.9)
- moved TP7 0.28 mm to (107.6, 43.9)
- moved AE1 0.18 mm to (98.5, 41.9)
- moved C14 0.16 mm to (107.0, 41.9)
- moved C19 0.10 mm to (99.3, 47.0)
- moved R15 0.10 mm to (99.3, 45.1)
Routing:
- net +4V: track 24.0 -> 27.9 mm
- net /WS2812_VDD: track 21.9 -> 25.5 mm
- net +3.3V: track 56.9 -> 59.6 mm, vias 20 -> 19
- net Net-(U8-OUTN): track 7.23 -> 9.43 mm
- net GND: track 104.7 -> 106.3 mm, vias 63 -> 62
- net /3V3_OUT: track 8.02 -> 9.11 mm
- net /SD_CMD: track 7.85 -> 8.72 mm
- net /I2C_SCL: track 10.1 -> 10.8 mm
- net /EXTIO_1: track 15.6 -> 16.2 mm
Other:
- outline, holes or cut-outs redrawn
- board text added: "0"
- board text added: "10"
- board text added: "12.2024"
- board text added: "@cbit"
- board text added: "B"
- board text added: "C"
- board text added: "G"
- board text added: "R"
- board text added: "V"
- board text added: "an"
- board text added: "rev 4"
- board text removed: "-"
- board text removed: "1 0"
- board text removed: "46"
- board text removed: "@cb1t"
- board text removed: "b1"
- board text removed: "b2"
- board text removed: "boot"
- board text removed: "rev3"
- board text removed: "rx"
- board text removed: "tx"
