File: pilkbrain.kicad_sch (KiCad schematic)
At the start: 101 parts, among them SW2 EVQPUC02K, SW3 EVQPUC02K, U1 ESP32-C3, U10 TS5A23157DGSR, U13 ESP32-S3, U3 SPX3819M5-L-3-3, U4 BQ24073RGT, U6 W25Q128JVS, U7 MT9700, U8 MAX98357AEWL+T, U9 MT9700, Y1 XO-40M, Y2 XO-32K

Commit message: before route
Parts:
- removed C10, C22: 10u, Capacitor_SMD:C_0603_1608Metric, symbol Device:C_Small
- removed C25, C3: 100n, Capacitor_SMD:C_0402_1005Metric, symbol Device:C_Small
- removed H1, H2, H3: M2, MountingHole:MountingHole_2.2mm_M2, symbol Mechanical:MountingHole
- removed PAD16: BAT+, Critbit_lib:diy_castellate_2.54, symbol Connector:TestPoint
- removed R12, R20, R26, R27, R28, R29: DNP/0603, Resistor_SMD:R_0603_1608Metric, symbol Device:R_Small
- removed R21, R22, R23, R25: 0R/0603, Resistor_SMD:R_0603_1608Metric, symbol Device:R_Small
- removed R30: 3k3/0603, Resistor_SMD:R_0603_1608Metric, symbol Device:R_Small
- removed U1: ESP32-C3, Package_DFN_QFN:QFN-32-1EP_5x5mm_P0.5mm_EP3.45x3.45mm, symbol Espressif:ESP32-C3
- removed U10: TS5A23157DGSR, easyeda2kicad:MSOP-10_L3.0-W3.0-P0.50-LS5.0-BL, symbol easyeda2kicad:TS5A23157DGSR
- removed U6: W25Q128JVS, Package_SO:SOIC-8_5.23x5.23mm_P1.27mm, symbol Memory_Flash:W25Q128JVS
- added C26, C29: 1u, Capacitor_SMD:C_0402_1005Metric, symbol Device:C_Small
- added C27, C30, C31: 100n, Capacitor_SMD:C_0402_1005Metric, symbol Device:C_Small
- added J1: USB_C_Receptacle_USB2.0, Connector_USB:USB_C_Receptacle_HRO_TYPE-C-31-M-12, symbol Connector:USB_C_Receptacle_USB2.0
- added J2: Conn_01x05, Connector_PinHeader_1.27mm:PinHeader_1x05_P1.27mm_Vertical, symbol Connector_Generic:Conn_01x05
- added PAD21, PAD22, PAD23, PAD24, PAD25, PAD26: BAT-, Critbit_lib:diy_castellate_2.54, symbol Connector:TestPoint
- added R31, R32, R33, R34, R6: 10k, Resistor_SMD:R_0402_1005Metric, symbol Device:R_Small
- added R35: 100k, Resistor_SMD:R_0402_1005Metric, symbol Device:R_Small
- added R36, R37: 5.1k, Resistor_SMD:R_0402_1005Metric, symbol Device:R_Small
- added U1: TF-123-ARP9H17, easyeda2kicad:TF-SMD_TF-123-ARP9H15, symbol easyeda2kicad:TF-123-ARP9H17
- C1: value 100n -> 10n
- C20: value 10u -> 1u; footprint Capacitor_SMD:C_0603_1608Metric -> Capacitor_SMD:C_0402_1005Metric; LCSC (none) -> C1525
- C23: value 10u -> 100n; footprint Capacitor_SMD:C_0603_1608Metric -> Capacitor_SMD:C_0402_1005Metric; LCSC (none) -> C1525
- R1: value 1k/0603 -> 3k3; footprint Resistor_SMD:R_0603_1608Metric -> Resistor_SMD:R_0402_1005Metric
- R2: value 100 -> 10k
- R4: value 3k3/0603 -> 3k3; footprint Resistor_SMD:R_0603_1608Metric -> Resistor_SMD:R_0402_1005Metric
- U13: footprint Package_DFN_QFN:QFN-56-1EP_7x7mm_P0.4mm_EP5.6x5.6mm -> Package_DFN_QFN:QFN-56-1EP_7x7mm_P0.4mm_EP4x4mm
- U5: footprint Critbit_lib:OLED_4Pin_128x32 -> Critbit_lib:OLED_4Pin_128x64_new
Connections:
- net +3.3V: now also C20.1, R1.2, R2.2, U13.20 (VDD3P3_RTC), U13.29 (VDD_SPI), U13.46 (VDD3P3_CPU), U13.55 (VDDA), U13.56 (VDDA), C26.1, C27.1, C29.1, C30.1, C31.1, R31.2, R32.2, R33.2, R34.2, R6.2, U1.4 (VDD)
- net 3V3_OUT: now also PAD19.1
- net BOOT_BUT1: now also U13.5 (GPIO0/BOOT), J2.2 (Pin_2)
- net EN_PERIPH: now also U13.15 (GPIO10/ADC1_CH9)
- net ESP_EN: now also U13.4 (CHIP_PU/RESET), J2.1 (Pin_1)
- net GND: now also PAD20.1, C26.2, C27.2, C29.2, C30.2, C31.2, J1.A1 (GND), J1.A12 (GND), J1.B1 (GND), J1.B12 (GND), J1.S1 (SHIELD), J2.3 (Pin_3), PAD23.1, R35.1, R36.1, R37.1, U1.6 (VSS)
- net I2C_SCL: now also PAD8.1, U13.7 (GPIO2/ADC1_CH1)
- net I2C_SDA: now also PAD9.1, R1.1, U13.8 (GPIO3/ADC1_CH2)
- net I2S_CLK: now also U13.12 (GPIO7/ADC1_CH6)
- net I2S_DAT: now also U13.11 (GPIO6/ADC1_CH5)
- net I2S_LRCLK: now also U13.10 (GPIO5/ADC1_CH4); no longer R2.1
- net USBDM: now also U13.25 (GPIO19/USB_D-/ADC2_CH8), J1.A7 (D-), J1.B7 (D-)
- net USBDP: now also U13.26 (GPIO20/USB_D+/ADC2_CH9), J1.A6 (D+), J1.B6 (D+)
- net VBUS: now also J1.A4 (VBUS), J1.A9 (VBUS), J1.B4 (VBUS), J1.B9 (VBUS)
- net VDD3P3: now also C23.1, L1.2
- net WS2812_OUT: now also U13.13 (GPIO8/ADC1_CH7), PAD22.1
- net WS2812_VDD: now also PAD21.1
- net at C5.1, Y2.1: now also U13.21 (GPIO15/ADC2_CH4/XTAL_32K_P)
- net at C6.1, Y2.2: now also U13.22 (GPIO16/ADC2_CH5/XTAL_32K_N)
- net at C7.1, Y1.1: now also U13.54 (XTAL_P)
- net at C8.1, Y1.3: now also U13.53 (XTAL_N)
- net BUT2: now reaches C18.1, R19.1, SW2.2, SW2.4
- net BUT2: no longer R1.1
- net at C35.1, L2.2: now also U13.1 (LNA_IN/RF)
- net TARG_TX: now reaches U13.49 (U0TXD/PROG/GPIO43)
- net TARG_TX: now also PAD14.1, J2.4 (Pin_4)
- net TARG_RX: now reaches U13.50 (U0RXD/PROG/GPIO44)
- net TARG_RX: now also PAD15.1, J2.5 (Pin_5)
- removed net TARG_RX_LRCLK: PAD15.1, R2.2
- removed net TARG_TX_B2: PAD14.1, R1.2
- new net: J1.B5 (CC2), R36.2
- new net: R35.2, U1.9 (SWITCH)
- new net: J1.A5 (CC1), R37.2
- new net SD_CLK: R31.1, U1.5 (CLK)
- new net SD_CMD: R32.1, U1.3 (CMD)
- new net SD_DAT0: R6.1, U1.7 (DAT0)
- new net SD_DAT1: R2.1, U1.8 (DAT1)
- new net SD_DAT2: R34.1, U1.1 (DAT2)
- new net SD_DAT3: R33.1, U1.2 (CD/DAT3)
- no-connect marks 4 -> 17
Other:
- note added: "(shared cap)"
- note added: "10u omitted"
- note added: "RTS DTR GND PRX PTX"
- moved on the sheet: AE1, C1, C2, C21, C24, C34, C35, C4, C5, C6, C7, C8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

Commit message: before move 4L
Parts:
- removed C31: 100n, Capacitor_SMD:C_0402_1005Metric, symbol Device:C_Small
- removed R15: 10k/0603, Resistor_SMD:R_0603_1608Metric, symbol Device:R_Small
- added R12: 10k, Resistor_SMD:R_0402_1005Metric, symbol Device:R_Small
Connections:
- net +3.3V: no longer R1.2, R4.2
- net 3V3_OUT: now also R1.2, R4.2
- net BOOT_BUT1: no longer PAD17.1
- net EN_PERIPH: now also U13.23 (GPIO17/ADC2_CH6); no longer U13.15 (GPIO10/ADC1_CH9)
- net GND: now also R12.1
- net I2C_SCL: now also U13.40 (GPIO35); no longer U13.7 (GPIO2/ADC1_CH1)
- net I2C_SDA: now also U13.42 (GPIO37); no longer U13.8 (GPIO3/ADC1_CH2)
- net I2S_CLK: now also U13.16 (GPIO11/ADC2_CH0); no longer U13.12 (GPIO7/ADC1_CH6)
- net I2S_DAT: now also U13.17 (GPIO12/ADC2_CH1); no longer U13.11 (GPIO6/ADC1_CH5)
- net I2S_LRCLK: now also U13.18 (GPIO13/ADC2_CH2); no longer U13.10 (GPIO5/ADC1_CH4)
- net SD_CLK: now also U13.39 (GPIO34)
- net SD_CMD: now also U13.27 (GPIO21)
- net SD_DAT0: now also U13.41 (GPIO36)
- net SD_DAT1: now also U13.43 (GPIO38)
- net SD_DAT2: now also U13.36 (SPICLK_N/GPIO48)
- net SD_DAT3: now also U13.24 (GPIO18/ADC2_CH7)
- net TARG_RX: no longer PAD15.1
- net TARG_TX: no longer PAD14.1
- net VBAT_MEAS: now also U13.15 (GPIO10/ADC1_CH9)
- net WS2812_OUT: now also U13.37 (SPICLK_P/GPIO47)
- net at PAD5.1, U4.1 (TS): now also R12.2
- net EN_3V3OUT: now reaches U13.19 (GPIO14/ADC2_CH3)
- net EN_3V3OUT: now also R18.2, U9.4 (EN)
Other:
- note added: "100n omitted"
- moved on the sheet: PAD18, PAD19, PAD20, PAD24, PAD25, PAD26, PAD8, PAD9, R1, R4

Commit message: DRC
Parts:
- added H1: M2, MountingHole:MountingHole_2.2mm_M2, symbol Mechanical:MountingHole
Connections:
- net BUT2: now also U13.13 (GPIO8/ADC1_CH7)
- net GND: now also PAD17.1; no longer PAD18.1
- net I2S_CLK: now also U13.18 (GPIO13/ADC2_CH2); no longer U13.16 (GPIO11/ADC2_CH0)
- net I2S_LRCLK: now also U13.16 (GPIO11/ADC2_CH0); no longer U13.18 (GPIO13/ADC2_CH2)
- net WS2812_OUT: no longer U13.13 (GPIO8/ADC1_CH7)
- net EXTIO_5: now reaches PAD25.1
- net EXTIO_5: now also U13.7 (GPIO2/ADC1_CH1)
- net EXTIO_3: now reaches PAD14.1
- net EXTIO_3: now also U13.9 (GPIO4/ADC1_CH3)
- net EXTIO_2: now reaches PAD15.1
- net EXTIO_2: now also U13.10 (GPIO5/ADC1_CH4)
- net EXTIO_4: now reaches PAD24.1
- net EXTIO_4: now also U13.8 (GPIO3/ADC1_CH2)
- net EXTIO_6: now reaches PAD26.1
- net EXTIO_6: now also U13.6 (GPIO1/ADC1_CH0)
- net EXTIO_1: now reaches U13.14 (GPIO9/ADC1_CH8)
- net EXTIO_1: now also PAD18.1
Other:
- moved on the sheet: PAD14, PAD15, PAD17, PAD18, PAD24, PAD25, PAD26

Commit message: before fab out
Parts:
- removed U2: ~, Critbit_lib:OLED_4Pin_64x48, symbol Critbit_lib:OLED_4Pin
- removed U5: ~, Critbit_lib:OLED_4Pin_128x64_new, symbol Critbit_lib:OLED_4Pin
- added C3: 1u, Capacitor_SMD:C_0402_1005Metric, symbol Device:C_Small
- added D1: LED_WHITE, LED_SMD:LED_0603_1608Metric, symbol Device:LED
- added L3: 24nH, Inductor_SMD:L_0402_1005Metric, symbol Device:L_Small
- added PAD16: 7, Critbit_lib:diy_castellate_2.54, symbol Connector:TestPoint
- added PAD27: 8, Critbit_lib:diy_castellate_2.54, symbol Connector:TestPoint
- added PAD28: 9, Critbit_lib:diy_castellate_2.54, symbol Connector:TestPoint
- added PAD29: 10, Critbit_lib:diy_castellate_2.54, symbol Connector:TestPoint
- added R15: 10k, Resistor_SMD:R_0402_1005Metric, symbol Device:R_Small
- AE1: LCSC (none) -> C127629
- C1: value 10n -> 100n
- C11, C12, C13, C14, C15, C16, C24, C32, C9: LCSC (none) -> C1691
- C17, C18, C19, C27, C33: LCSC (none) -> C1525
- C20, C26, C29: LCSC C1525 -> C14445
- C21: value 100n -> 1u; LCSC (none) -> C14445
- C34, C35: value 100n -> 3.3p
- C5, C6, C7, C8: value 20p(TBD) -> 12p; LCSC C1525 -> C76700
- D3: LCSC (none) -> C2290
- D4: LCSC (none) -> C2286
- J1: LCSC (none) -> C165948
- L1: value 2nH -> 2nH/500mA; LCSC (none) -> C97984
- L2: value TBD -> 2nH/500mA; LCSC (none) -> C97984
- PAD11: value BAT- -> EN_3V3
- PAD12: value BAT- -> 5V
- PAD13, PAD20, PAD23: value BAT- -> GND
- PAD14: value BAT+ -> 3
- PAD15: value BAT+ -> 2
- PAD17: value BAT+ -> GND
- PAD18: value BAT+ -> 1
- PAD19: value BAT- -> 3V3_OUT
- PAD21: value BAT- -> 4V_OUT
- PAD22: value BAT- -> WS2812_OUT
- PAD24: value BAT- -> 4
- PAD25: value BAT- -> 5
- PAD26: value BAT- -> 6
- PAD6: value BAT- -> DM
- PAD7: value BAT- -> DP
- PAD8: value BAT- -> SCL
- PAD9: value BAT- -> SDA
- R1, R4: value 3k3 -> 2k
- R13, R14: value 3k -> 2k
- SW2, SW3: LCSC (none) -> C79174; LCSC Part C79174 -> (none)
- U1: LCSC (none) -> C2982548; LCSC Part C2982548 -> (none)
- U13: LCSC (none) -> C2913196
- U3: LCSC (none) -> C9055
- U4: LCSC (none) -> C15220
- U7, U9: LCSC (none) -> C89855; LCSC Part C89855 -> (none)
- U8: LCSC (none) -> C2682619; LCSC Part C2682619 -> (none)
- Y1: LCSC (none) -> C431168
- Y2: LCSC (none) -> C5366532
Connections:
- net EN_LEFT is gone; now on net EN_PERIPH: PAD10.1
- net EN_RIGHT is gone; now on net EN_3V3OUT: PAD11.1
- net +3.3V: now also D3.2 (A), D4.2 (A), C3.1
- net +4V: now also U3.3 (EN); no longer D3.2 (A), D4.2 (A)
- net BQ_PGOOD: now also U13.51 (GPIO45)
- net GND: now also C3.2, R15.1
- net at C7.1, Y1.1: now also L3.1; no longer U13.54 (XTAL_P)
- net EXTIO_10: now reaches U13.44 (MTCK/JTAG/GPIO39)
- net EXTIO_10: now also PAD29.1
- net EXTIO_8: now reaches U13.45 (MTDO/JTAG/GPIO40)
- net EXTIO_8: now also PAD27.1
- net EXTIO_7: now reaches U13.47 (MTDI/JTAG/GPIO41)
- net EXTIO_7: now also PAD16.1
- net EXTIO_9: now reaches U13.48 (MTMS/JTAG/GPIO42)
- net EXTIO_9: now also PAD28.1
- net LED_STA: now reaches U13.52 (GPIO46)
- net LED_STA: now also D1.2 (A)
- new net: D1.1 (K), R15.2
- new net: L3.2, U13.54 (XTAL_P)
Other:
- note removed: "C2290"
- note removed: "C84256"
- moved on the sheet: AE1, C1, C11, C12, C13, C14, C15, C16, C17, C18, C19, C2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

Commit message: order(?)
Parts:
- C20, C21, C26, C29, C3: LCSC C14445 -> C52923
- C34, C35: LCSC C1525 -> C1565
- C5, C6, C7, C8: LCSC C76700 -> C1547
Changed lines of the file:
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@@
 	(text "s3 - 2.2\ns3FH8 - 3.0\nc3fh4 - 1.4\nc3 - 1.2\n16M - 0.3-0.5\n\nS3@8 - 3.0\nS3@16 - 2.5\nc3@16 - 1.5"
 		(exclude_from_sim no)
-		(at 307.848 20.32 0)
+		(at 222.504 25.146 0)
 		(effects
 			(font
 				(size 1.27 1.27)
 			)
+			(justify left)
 		)
 	)
@@
 			)
 		)
-		(property "LCSC" "C1525"
+		(property "LCSC" "C1565"
 			(at 50.8 99.06 0)
 			(effects
@@
 			)
 		)
-		(property "LCSC" "C14445"
+		(property "LCSC" "C52923"
 			(at 142.24 99.06 0)
 			(effects
@@
 				)
 				(justify left)
-				(hide yes)
 			)
 		)
@@
 			)
 		)
-		(property "LCSC" "C14445"
+		(property "LCSC" "C52923"
 			(at 147.32 85.09 0)
 			(effects
@@
 			)
 		)
-		(property "LCSC" "C76700"
+		(property "LCSC" "C1547"
 			(at 74.93 129.54 0)
 			(effects
@@
 			)
 		)
-		(property "LCSC" "C1525"
+		(property "LCSC" "C1565"
 			(at 59.69 99.06 0)
 			(effects
@@
 			)
 		)
-		(property "LCSC" "C14445"
+		(property "LCSC" "C52923"
 			(at 96.52 99.06 0)
 			(effects
@@
 			)
 		)
-		(property "LCSC" "C14445"
+		(property "LCSC" "C52923"
 			(at 40.64 113.03 0)
 			(effects
@@
 			)
 		)
-		(property "LCSC" "C76700"
+		(property "LCSC" "C1547"
 			(at 54.61 119.38 0)
 			(effects
@@
 			)
 		)
-		(property "LCSC" "C76700"
+		(property "LCSC" "C1547"
 			(at 74.93 119.38 0)
 			(effects
@@
 			)
 		)
-		(property "LCSC" "C14445"
+		(property "LCSC" "C52923"
 			(at 87.63 90.17 0)
 			(effects
@@
 			)
 		)
-		(property "LCSC" "C76700"
+		(property "LCSC" "C1547"
 			(at 54.61 129.54 0)
 			(effects

Commit message: new formfactor placement etc
Parts:
- removed C20: 1u, Capacitor_SMD:C_0402_1005Metric, symbol Device:C_Small
- removed C24: 10u, Capacitor_SMD:C_0603_1608Metric, symbol Device:C_Small
- removed C27: 100n, Capacitor_SMD:C_0402_1005Metric, symbol Device:C_Small
- removed D1, D3: LED_WHITE, LED_SMD:LED_0603_1608Metric, symbol Device:LED
- removed D4: LED_RED, LED_SMD:LED_0603_1608Metric, symbol Device:LED
- removed H1: M2, MountingHole:MountingHole_2.2mm_M2, symbol Mechanical:MountingHole
- removed PAD10: BAT-, Critbit_lib:diy_castellate_2.54, symbol Connector:TestPoint
- removed PAD11: EN_3V3, Critbit_lib:diy_castellate_2.54, symbol Connector:TestPoint
- removed PAD28: 9, Critbit_lib:diy_castellate_2.54, symbol Connector:TestPoint
- removed PAD29: 10, Critbit_lib:diy_castellate_2.54, symbol Connector:TestPoint
- removed R12, R31, R32, R33, R34, R6: 10k, Resistor_SMD:R_0402_1005Metric, symbol Device:R_Small
- removed R35: 100k, Resistor_SMD:R_0402_1005Metric, symbol Device:R_Small
- removed U1: TF-123-ARP9H17, easyeda2kicad:TF-SMD_TF-123-ARP9H15, symbol easyeda2kicad:TF-123-ARP9H17
- added C10: 10u, Capacitor_SMD:C_0603_1608Metric, symbol Device:C_Small
- added CN3: YXT-BB10-24S-02, easyeda2kicad:CONN-SMD_YXT-BB10-24S-02, symbol easyeda2kicad:YXT-BB10-24S-02
- added U1: ~, Critbit_lib:OLED_4Pin_128x64_new, symbol Critbit_lib:OLED_4Pin
- added U2, U5, U6: XL-1005UWC_C20613596, easyeda2kicad:LED0402-RD_YELLOW, symbol easyeda2kicad:XL-1005UWC_C20613596
- C14: value 10u -> 1u; footprint Capacitor_SMD:C_0603_1608Metric -> Capacitor_SMD:C_0402_1005Metric; LCSC C1691 -> C52923
- PAD3, PAD4: value TP -> 10
- R16: value 500k -> 510k/0603; footprint Resistor_SMD:R_0402_1005Metric -> Resistor_SMD:R_0603_1608Metric
- R2: value 10k -> 10k/DNP; footprint Resistor_SMD:R_0402_1005Metric -> Resistor_SMD:R_0603_1608Metric
- R3, R5: value 100k -> 10k
Connections:
- net +3.3V: now also U5.2 (A), U6.2 (A); no longer R2.2
- net +4V: now also C10.1
- net 3V3_OUT: now also CN3.20, CN3.21
- net BQ_CHG: now also U13.44 (MTCK/JTAG/GPIO39)
- net BQ_PGOOD: now also U13.43 (GPIO38); no longer U13.51 (GPIO45)
- net BUT2: now also U13.48 (MTMS/JTAG/GPIO42); no longer U13.13 (GPIO8/ADC1_CH7)
- net EN_3V3OUT: now also U13.12 (GPIO7/ADC1_CH6); no longer U13.19 (GPIO14/ADC2_CH3)
- net EXTIO_1: now also U13.11 (GPIO6/ADC1_CH5); no longer U13.14 (GPIO9/ADC1_CH8)
- net EXTIO_10: no longer U13.44 (MTCK/JTAG/GPIO39)
- net EXTIO_3: now also U13.19 (GPIO14/ADC2_CH3); no longer U13.9 (GPIO4/ADC1_CH3)
- net EXTIO_4: now also U13.18 (GPIO13/ADC2_CH2); no longer U13.8 (GPIO3/ADC1_CH2)
- net EXTIO_5: now also U13.17 (GPIO12/ADC2_CH1); no longer U13.7 (GPIO2/ADC1_CH1)
- net EXTIO_6: now also U13.16 (GPIO11/ADC2_CH0); no longer U13.6 (GPIO1/ADC1_CH0)
- net EXTIO_7: now also U13.15 (GPIO10/ADC1_CH9); no longer U13.47 (MTDI/JTAG/GPIO41)
- net EXTIO_8: now also U13.14 (GPIO9/ADC1_CH8); no longer U13.45 (MTDO/JTAG/GPIO40)
- net EXTIO_9: no longer U13.48 (MTMS/JTAG/GPIO42)
- net GND: now also R2.1, C10.2, CN3.10, CN3.12, CN3.2, CN3.24, CN3.25, CN3.26, CN3.27, CN3.28, CN3.4, CN3.6, CN3.8
- net I2C_SCL: now also CN3.19; no longer U13.40 (GPIO35)
- net I2C_SDA: now also CN3.18; no longer U13.42 (GPIO37)
- net I2S_CLK: now also U13.45 (MTDO/JTAG/GPIO40); no longer U13.18 (GPIO13/ADC2_CH2)
- net I2S_DAT: now also U13.47 (MTDI/JTAG/GPIO41); no longer U13.17 (GPIO12/ADC2_CH1)
- net I2S_LRCLK: now also U13.51 (GPIO45); no longer U13.16 (GPIO11/ADC2_CH0)
- net LED_STA: now also U13.13 (GPIO8/ADC1_CH7), U2.2 (A); no longer U13.52 (GPIO46)
- net SD_CLK: now also U13.38 (GPIO33), CN3.5; no longer U13.39 (GPIO34)
- net SD_CMD: now also U13.39 (GPIO34), CN3.7; no longer U13.27 (GPIO21)
- net SD_DAT0: now also U13.40 (GPIO35), CN3.3; no longer U13.41 (GPIO36)
- net SD_DAT1: now also U13.41 (GPIO36), CN3.1; no longer R2.1, U13.43 (GPIO38)
- net SD_DAT2: now also U13.37 (SPICLK_P/GPIO47), CN3.11; no longer U13.36 (SPICLK_N/GPIO48)
- net SD_DAT3: now also U13.36 (SPICLK_N/GPIO48), CN3.9; no longer U13.24 (GPIO18/ADC2_CH7)
- net USBDM: now also CN3.23
- net USBDP: now also CN3.22
- net VBAT_MEAS: now also U13.24 (GPIO18/ADC2_CH7); no longer U13.15 (GPIO10/ADC1_CH9)
- net WS2812_OUT: now also U13.27 (GPIO21); no longer U13.37 (SPICLK_P/GPIO47)
- net WS2812_VDD: now also CN3.13, CN3.14
- net at R9.2: now also U5.1 (K)
- net at PAD5.1, U4.1 (TS): now also R2.2
- net at R15.2: now also U2.1 (K)
- net at R8.2: now also U6.1 (K)
- new net SD_DET: CN3.17, U13.42 (GPIO37)
- no-connect marks 17 -> 13
Other:
- note added: "1u omitted"
- note added: "shared cap"
- note removed: "(shared cap)"
- note removed: "10u omitted"

Commit message: rev2 prod?
Parts:
- removed J1: USB_C_Receptacle_USB2.0, Connector_USB:USB_C_Receptacle_HRO_TYPE-C-31-M-12, symbol Connector:USB_C_Receptacle_USB2.0
- removed R36, R37: 5.1k, Resistor_SMD:R_0402_1005Metric, symbol Device:R_Small
- removed U1: ~, Critbit_lib:OLED_4Pin_128x64_new, symbol Critbit_lib:OLED_4Pin
- added R12, R6: 5.1k, Resistor_SMD:R_0402_1005Metric, symbol Device:R_Small
- added USB1: GT-USB-7055E, easyeda2kicad:USB-C-SMD_GT-USB-7055E, symbol easyeda2kicad:GT-USB-7055E
- CN3: LCSC (none) -> C2763965; LCSC Part C2763965 -> (none)
- U2, U5, U6: LCSC (none) -> C20613596; LCSC Part C20613596 -> (none)
Connections:
- net +3.3V: now also CN3.15, CN3.16
- net 3V3_OUT: no longer CN3.20, CN3.21
- net EN_PERIPH: now also U13.16 (GPIO11/ADC2_CH0); no longer U13.23 (GPIO17/ADC2_CH6)
- net EXTIO_6: now also U13.7 (GPIO2/ADC1_CH1); no longer U13.16 (GPIO11/ADC2_CH0)
- net GND: now also R12.2, R6.2, USB1.0 (SHELL), USB1.A1 (GND), USB1.A12 (GND), USB1.B1 (GND), USB1.B12 (GND)
- net I2C_SCL: now also CN3.18, U13.45 (MTDO/JTAG/GPIO40); no longer CN3.19
- net I2C_SDA: now also CN3.19, U13.47 (MTDI/JTAG/GPIO41); no longer CN3.18
- net I2S_CLK: now also U13.37 (SPICLK_P/GPIO47); no longer U13.45 (MTDO/JTAG/GPIO40)
- net I2S_DAT: now also U13.23 (GPIO17/ADC2_CH6); no longer U13.47 (MTDI/JTAG/GPIO41)
- net SD_DAT2: now also U13.27 (GPIO21); no longer U13.37 (SPICLK_P/GPIO47)
- net SD_DET: now also U13.8 (GPIO3/ADC1_CH2); no longer U13.42 (GPIO37)
- net USBDM: now also USB1.A7 (D-), USB1.B7 (D-)
- net USBDP: now also USB1.A6 (D+), USB1.B6 (D+)
- net VBUS: now also CN3.20, CN3.21, USB1.A4 (VBUS), USB1.A9 (VBUS), USB1.B4 (VBUS), USB1.B9 (VBUS)
- net WS2812_OUT: now also U13.9 (GPIO4/ADC1_CH3); no longer U13.27 (GPIO21)
- net at U8.A3 (OUTP): now also PAD3.1; no longer PAD4.1
- net at U8.B3 (OUTN): now also PAD4.1; no longer PAD3.1
- new net: R12.1, USB1.B5 (CC2)
- new net: R6.1, USB1.A5 (CC1)
Other:
- note added: "C7450622"
- moved on the sheet: PAD3, PAD4
