File: pilkbrain.kicad_sch (KiCad schematic)
At the start: 93 parts, among them CN3 YXT-BB10-24S-02, J2 Conn_01x05, SW2 EVQPUC02K, SW3 EVQPUC02K, U13 ESP32-S3, U2 XL-1005UWC_C20613596, U3 SPX3819M5-L-3-3, U4 BQ24073RGT, U5 XL-1005UWC_C20613596, U6 XL-1005UWC_C20613596, U7 MT9700, U8 MAX98357AEWL+T, U9 MT9700, Y1 XO-40M, Y2 XO-32K

Commit message: 3rd redo but good this time
Parts:
- removed C26: 1u, Capacitor_SMD:C_0402_1005Metric, symbol Device:C_Small
- removed C32: 10u, Capacitor_SMD:C_0603_1608Metric, symbol Device:C_Small
- removed CN3: YXT-BB10-24S-02, easyeda2kicad:CONN-SMD_YXT-BB10-24S-02, symbol easyeda2kicad:YXT-BB10-24S-02
- removed J2: Conn_01x05, Connector_PinHeader_1.27mm:PinHeader_1x05_P1.27mm_Vertical, symbol Connector_Generic:Conn_01x05
- removed PAD22: WS2812_OUT, Critbit_lib:diy_castellate_2.54, symbol Connector:TestPoint
- removed PAD23: GND, Critbit_lib:diy_castellate_2.54, symbol Connector:TestPoint
- removed SW2, SW3: EVQPUC02K, easyeda2kicad:SW-SMD_EVQPUD02K, symbol easyeda2kicad:EVQPUC02K
- removed U3: SPX3819M5-L-3-3, Package_TO_SOT_SMD:SOT-23-5, symbol Regulator_Linear:SPX3819M5-L-3-3
- removed U7, U9: MT9700, easyeda2kicad:SOT-23-5_L3.0-W1.7-P0.95-LS2.8-BR, symbol easyeda2kicad:MT9700
- removed USB1: GT-USB-7055E, easyeda2kicad:USB-C-SMD_GT-USB-7055E, symbol easyeda2kicad:GT-USB-7055E
- added C20, C24: 100n, Capacitor_SMD:C_0402_1005Metric, symbol Device:C_Small
- added C22: 10u, Capacitor_SMD:C_0402_1005Metric, symbol Device:C_Small
- added CN1: SM02B-SRSS-TB (LF)(SN), easyeda2kicad:CONN-SMD_2P-P1.00_SM02B-SRSS-TB-LF-SN, symbol easyeda2kicad:SM02B-SRSS-TB(LF)(SN)
- added PAD10, PAD11, PAD28: PAD_T, Critbit_lib:diy_castellate_tight, symbol Connector:TestPoint
- added R20, R21, R22, R23, R25: 10k, Resistor_SMD:R_0402_1005Metric, symbol Device:R_Small
- added R26: 100k, Resistor_SMD:R_0402_1005Metric, symbol Device:R_Small
- added SW1, SW3: TS24CA, easyeda2kicad:SW-SMD_TS24CA, symbol easyeda2kicad:TS24CA
- added U1: TYPE-C 16P LTH8.8, easyeda2kicad:USB-C-SMD_TYPE-C-16P-LTH8.8, symbol easyeda2kicad:TYPE-C16PLTH8.8
- added U10: A-SP1102AR6GHC-A01-2C, easyeda2kicad:LED-SMD_4P-L3.0-W1.5_A-SP1102AR6GHC-A01-2C, symbol easyeda2kicad:A-SP1102AR6GHC-A01-2C
- added U11: TF-123-ARP9H17, easyeda2kicad:TF-SMD_TF-123-ARP9H15, symbol easyeda2kicad:TF-123-ARP9H17
- added U12: SM03B-SRSS-TB(LF)(SN)(P), easyeda2kicad:CONN-SMD_SM03B-SRSS-TB-LF-SN-P, symbol easyeda2kicad:SM03B-SRSS-TB(LF)(SN)(P)
- added U3, U9: SSP7615-33DFR, easyeda2kicad:DFN-4_L1.0-W1.0-P0.65-BL-EP, symbol easyeda2kicad:SSP7615-33DFR
- added U7: AP2552FDC-7, easyeda2kicad:WDFN-6_L2.0-W2.0-P0.65-BL-EP-1, symbol easyeda2kicad:AP2552FDC-7
- C10, C12, C15: value 10u -> 1u; footprint Capacitor_SMD:C_0603_1608Metric -> Capacitor_SMD:C_0402_1005Metric; LCSC C1691 -> C52923
- C11: value 10u -> 47uF/0805; footprint Capacitor_SMD:C_0603_1608Metric -> Capacitor_SMD:C_0805_2012Metric; LCSC C1691 -> C15525
- C13, C16, C9: footprint Capacitor_SMD:C_0603_1608Metric -> Capacitor_SMD:C_0402_1005Metric; LCSC C1691 -> C15525
- PAD1: value BAT- -> PAD_T; footprint Critbit_lib:diy_castellate_2.54 -> Critbit_lib:diy_castellate_tight
- PAD12: value 5V -> PAD_T; footprint Critbit_lib:diy_castellate_2.54 -> Critbit_lib:diy_castellate_tight
- PAD13, PAD17: value GND -> PAD_T; footprint Critbit_lib:diy_castellate_2.54 -> Critbit_lib:diy_castellate_tight
- PAD14: value 3 -> PAD_T; footprint Critbit_lib:diy_castellate_2.54 -> Critbit_lib:diy_castellate_tight
- PAD15: value 2 -> PAD_T; footprint Critbit_lib:diy_castellate_2.54 -> Critbit_lib:diy_castellate_tight
- PAD16: value 7 -> PAD_T; footprint Critbit_lib:diy_castellate_2.54 -> Critbit_lib:diy_castellate_tight
- PAD18: value 1 -> PAD_T; footprint Critbit_lib:diy_castellate_2.54 -> Critbit_lib:diy_castellate_tight
- PAD19: value 3V3_OUT -> PAD
- PAD2: value BAT+ -> PAD_T; footprint Critbit_lib:diy_castellate_2.54 -> Critbit_lib:diy_castellate_tight
- PAD20: value GND -> PAD
- PAD21: value 4V_OUT -> PAD
- PAD24: value 4 -> PAD_T; footprint Critbit_lib:diy_castellate_2.54 -> Critbit_lib:diy_castellate_tight
- PAD25: value 5 -> PAD_T; footprint Critbit_lib:diy_castellate_2.54 -> Critbit_lib:diy_castellate_tight
- PAD26: value 6 -> PAD_T; footprint Critbit_lib:diy_castellate_2.54 -> Critbit_lib:diy_castellate_tight
- PAD27: value 8 -> PAD_T; footprint Critbit_lib:diy_castellate_2.54 -> Critbit_lib:diy_castellate_tight
- PAD3, PAD4: value 10 -> PAD_T; footprint Critbit_lib:diy_castellate_2.54 -> Critbit_lib:diy_castellate_tight
- PAD5: value TC -> PAD_T; footprint Critbit_lib:diy_castellate_2.54 -> Critbit_lib:diy_castellate_tight
- PAD6: value DM -> PAD_T; footprint Critbit_lib:diy_castellate_2.54 -> Critbit_lib:diy_castellate_tight
- PAD7: value DP -> PAD_T; footprint Critbit_lib:diy_castellate_2.54 -> Critbit_lib:diy_castellate_tight
- PAD8: value SCL -> PAD
- PAD9: value SDA -> PAD
- R10: value 10k -> 100k
- U13: footprint Package_DFN_QFN:QFN-56-1EP_7x7mm_P0.4mm_EP4x4mm -> Package_DFN_QFN:QFN-56-1EP_7x7mm_P0.4mm_EP5.6x5.6mm; LCSC C2913196 -> C3013940
- Y1: footprint Crystal:Crystal_SMD_3225-4Pin_3.2x2.5mm -> Crystal:Crystal_SMD_2520-4Pin_2.5x2.0mm; LCSC C431168 -> C2885592
- Y2: footprint Crystal:Crystal_SMD_3215-2Pin_3.2x1.5mm -> Crystal:Crystal_SMD_2012-2Pin_2.0x1.2mm; LCSC C5366532 -> C7500573
Connections:
- net +3.3V: now also R17.2, C22.1, C24.1, R20.2, R21.2, R22.2, R23.2, R25.2, U11.4 (VDD), U9.1 (VOUT); no longer C14.1
- net +4V: now also C13.1, C14.1, C20.1, U3.4 (VIN), U7.6 (IN), U9.3 (EN), U9.4 (VIN); no longer C11.1
- net 3V3_OUT: now also U3.1 (VOUT)
- net BOOT_BUT1: now also SW1.4
- net BUT2: now also SW3.4
- net EN_3V3OUT: now also U3.3 (EN)
- net EN_PERIPH: now also U7.4 (EN)
- net GND: now also C20.2, C22.2, C24.2, R26.1, SW1.1, SW1.22 (2), SW1.3, SW3.1, SW3.22 (2), SW3.3, U1.13 (GND), U1.14 (GND), U1.15 (GND), U1.16 (GND), U1.A1 (GND), U1.A12 (GND), U1.B1 (GND), U1.B12 (GND), U11.6 (VSS), U12.3, U12.4, U12.5, U3.2 (GND), U7.5 (GND), U7.7 (EXP), U9.2 (GND); no longer PAD1.1, PAD17.1, R17.1
- net I2S_CLK: no longer U13.37 (SPICLK_P/GPIO47)
- net LIPO+: now also C11.1, U12.1; no longer C13.1, PAD2.1
- net SD_CLK: now also R21.1, U11.5 (CLK)
- net SD_CMD: now also U13.41 (GPIO36), R22.1, U11.3 (CMD); no longer U13.39 (GPIO34)
- net SD_DAT0: now also U13.39 (GPIO34), R20.1, U11.7 (DAT0); no longer U13.40 (GPIO35)
- net SD_DAT1: now also R17.1, U13.40 (GPIO35), U11.8 (DAT1); no longer U13.41 (GPIO36)
- net SD_DAT2: now also R25.1, U11.1 (DAT2)
- net SD_DAT3: now also R23.1, U11.2 (CD/DAT3)
- net SD_DET: now also U13.37 (SPICLK_P/GPIO47), R26.2, U11.9 (SWITCH); no longer U13.8 (GPIO3/ADC1_CH2)
- net USBDM: now also U1.A7 (D-), U1.B7 (D-)
- net USBDP: now also U1.A6 (D+), U1.B6 (D+)
- net VBUS: now also U1.A4 (VBUS), U1.A9 (VBUS), U1.B4 (VBUS), U1.B9 (VBUS)
- net WS2812_VDD: now also U7.1 (OUT)
- net at R2.2, U4.1 (TS): now also U12.2; no longer PAD5.1
- net at U8.A3 (OUTP): now also CN1.2; no longer PAD3.1
- net at U8.B3 (OUTN): now also CN1.1; no longer PAD4.1
- net at R10.2: now also U7.2 (ILIM)
- net at R12.1: now also U1.B5 (CC2)
- net at R6.1: now also U1.A5 (CC1)
- new net EXTIO_10: PAD11.1
- new net EXTIO_11: PAD28.1
- new net EXTIO_12: PAD1.1
- new net EXTIO_13: PAD2.1
- new net EXTIO_14: PAD3.1
- new net EXTIO_15: PAD4.1
- new net EXTIO_16: PAD5.1
- new net EXTIO_17: PAD17.1
- new net EXTIO_9: PAD10.1
- no-connect marks 13 -> 18
Other:
- note added: "Coincell footprint for the future C70373"
- note added: "TODO GLITCH!!!!!!"
- note added: "omitted"
- note added: "~250mA"
- note removed: "RTS DTR GND PRX PTX"
- note removed: "~500mA"
- moved on the sheet: C11, C13, C17, C19, PAD14, PAD15, PAD16, PAD18, PAD24, PAD25, PAD26, PAD27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
