File: pilkbrain.kicad_sch (KiCad schematic)
At the start: 103 parts, among them CN1 SM02B-SRSS-TB (LF)(SN), SW1 TS24CA, SW3 TS24CA, U1 TYPE-C 16P LTH8.8, U10 A-SP1102AR6GHC-A01-2C, U11 TF-123-ARP9H17, U12 SM03B-SRSS-TB(LF)(SN)(P), U13 ESP32-S3, U2 XL-1005UWC_C20613596, U3 SSP7615-33DFR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

Commit message: before order
Parts:
- removed PAD17, PAD5: PAD_T, Critbit_lib:diy_castellate_tight, symbol Connector:TestPoint
- removed U10: A-SP1102AR6GHC-A01-2C, easyeda2kicad:LED-SMD_4P-L3.0-W1.5_A-SP1102AR6GHC-A01-2C, symbol easyeda2kicad:A-SP1102AR6GHC-A01-2C
- added R27: 47k, Resistor_SMD:R_0402_1005Metric, symbol Device:R_Small
- added TP1, TP10, TP11, TP7, TP9: TP, TestPoint:TestPoint_Pad_D1.0mm, symbol Connector:TestPoint
- C11: LCSC C15525 -> C16780
- C24: LCSC (none) -> C1525
- C3: value 1u -> 10u; LCSC C52923 -> C15525
- CN1: LCSC (none) -> C160402; LCSC Part C160402 -> (none)
- R10, R26: value 100k -> 47k
- R16: value 510k/0603 -> 510k
- SW1, SW3: LCSC (none) -> C393942; LCSC Part C393942 -> (none)
- U1: LCSC (none) -> C5187469; LCSC Part C5187469 -> (none)
- U11: LCSC (none) -> C2982548; LCSC Part C2982548 -> (none)
- U12: LCSC (none) -> C160403; LCSC Part C160403 -> (none)
Connections:
- net EXTIO_11 is gone; now on net BQ_CHG: PAD28.1
- net EXTIO_12 is gone; now on net BQ_PGOOD: PAD1.1
- net EXTIO_13 is gone; now on net BOOT_BUT1: PAD2.1
- net EXTIO_14 is gone; now on net TARG_TX: PAD3.1
- net EXTIO_15 is gone; now on net TARG_RX: PAD4.1
- net WS2812_OUT is gone; now on net EXTIO_10: U13.9 (GPIO4/ADC1_CH3)
- net 3V3_OUT: now also R27.2
- net EN_3V3OUT: now also U13.8 (GPIO3/ADC1_CH2); no longer U13.12 (GPIO7/ADC1_CH6)
- net EN_PERIPH: now also U13.23 (GPIO17/ADC2_CH6); no longer U13.16 (GPIO11/ADC2_CH0)
- net ESP_EN: now also TP7.1
- net EXTIO_1: now also U13.27 (GPIO21); no longer U13.11 (GPIO6/ADC1_CH5)
- net EXTIO_2: now also U13.47 (MTDI/JTAG/GPIO41); no longer U13.10 (GPIO5/ADC1_CH4)
- net EXTIO_3: now also U13.24 (GPIO18/ADC2_CH7); no longer U13.19 (GPIO14/ADC2_CH3)
- net EXTIO_4: now also U13.51 (GPIO45); no longer U13.18 (GPIO13/ADC2_CH2)
- net EXTIO_5: now also U13.19 (GPIO14/ADC2_CH3); no longer U13.17 (GPIO12/ADC2_CH1)
- net EXTIO_6: now also U13.18 (GPIO13/ADC2_CH2); no longer U13.7 (GPIO2/ADC1_CH1)
- net EXTIO_7: now also U13.17 (GPIO12/ADC2_CH1); no longer U13.15 (GPIO10/ADC1_CH9)
- net EXTIO_8: now also U13.10 (GPIO5/ADC1_CH4); no longer U13.14 (GPIO9/ADC1_CH8)
- net EXTIO_9: now also U13.11 (GPIO6/ADC1_CH5)
- net GND: now also CN1.3, CN1.4, SW1.2, SW3.2, U3.5 (EP), U9.5 (EP), TP1.1; no longer SW1.22 (2), SW3.22 (2)
- net I2C_SCL: now also U13.7 (GPIO2/ADC1_CH1); no longer U13.45 (MTDO/JTAG/GPIO40)
- net I2C_SDA: now also U13.6 (GPIO1/ADC1_CH0); no longer U13.47 (MTDI/JTAG/GPIO41)
- net I2S_CLK: now also U13.12 (GPIO7/ADC1_CH6), TP9.1
- net I2S_DAT: now also U13.14 (GPIO9/ADC1_CH8), TP11.1; no longer U13.23 (GPIO17/ADC2_CH6)
- net I2S_LRCLK: now also U13.16 (GPIO11/ADC2_CH0), TP10.1; no longer U13.51 (GPIO45)
- net LED_STA: now also U13.45 (MTDO/JTAG/GPIO40); no longer U13.13 (GPIO8/ADC1_CH7)
- net SD_CLK: now also U13.40 (GPIO35); no longer U13.38 (GPIO33)
- net SD_CMD: now also U13.38 (GPIO33); no longer U13.41 (GPIO36)
- net SD_DAT0: now also U13.41 (GPIO36); no longer U13.39 (GPIO34)
- net SD_DAT1: now also U13.42 (GPIO37); no longer U13.40 (GPIO35)
- net SD_DAT2: now also U13.36 (SPICLK_N/GPIO48); no longer U13.27 (GPIO21)
- net SD_DAT3: now also U13.37 (SPICLK_P/GPIO47); no longer U13.36 (SPICLK_N/GPIO48)
- net SD_DET: now also U13.39 (GPIO34); no longer U13.37 (SPICLK_P/GPIO47)
- net VBAT_MEAS: now also U13.13 (GPIO8/ADC1_CH7); no longer U13.24 (GPIO18/ADC2_CH7)
- net PERIPH_FAULT: now reaches U7.3 (~{FAULT})
- net PERIPH_FAULT: now also U13.15 (GPIO10/ADC1_CH9)
- net at U8.A3 (OUTP): now also CN1.1; no longer CN1.2
- net at U8.B3 (OUTN): now also CN1.2; no longer CN1.1
- net 3V3_MEAS: now reaches U13.52 (GPIO46)
- net 3V3_MEAS: now also R27.1
- no-connect marks 18 -> 16
Other:
- note added: "datasheet not specified if connect needed"
- note added: "put AP2553 low-level glitch on io17"
- note added: "~500mA"
- note removed: "TODO GLITCH!!!!!!"
- note removed: "~250mA"
- moved on the sheet: PAD1, PAD2, PAD28, PAD3, PAD4

Commit message: another element swappage
Parts:
- U7: LCSC C150475 -> C211419
Connections:
- net EXTIO_8: now also U13.12 (GPIO7/ADC1_CH6); no longer U13.10 (GPIO5/ADC1_CH4)
- net EXTIO_9: now also U13.10 (GPIO5/ADC1_CH4); no longer U13.11 (GPIO6/ADC1_CH5)
- net I2S_CLK: now also U13.11 (GPIO6/ADC1_CH5); no longer U13.12 (GPIO7/ADC1_CH6)
Changed lines of the file:
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@@
 	)
 	(label "EXTIO_8"
-		(at 152.4 135.89 0)
+		(at 152.4 140.97 0)
 		(fields_autoplaced yes)
 		(effects
@@
 	)
 	(label "I2S_CLK"
-		(at 152.4 140.97 0)
+		(at 152.4 138.43 0)
 		(fields_autoplaced yes)
 		(effects
@@
 	)
 	(label "EXTIO_9"
-		(at 152.4 138.43 0)
+		(at 152.4 135.89 0)
 		(fields_autoplaced yes)
 		(effects
@@
 			)
 		)
-		(property "LCSC" "C150475"
+		(property "LCSC" "C211419"
 			(at 187.96 72.39 0)
 			(effects

Commit message: finish route?
Parts:
- removed C18: 100n, Capacitor_SMD:C_0402_1005Metric, symbol Device:C_Small
- removed R19: 10k, Resistor_SMD:R_0402_1005Metric, symbol Device:R_Small
- removed SW3: TS24CA, easyeda2kicad:SW-SMD_TS24CA, symbol easyeda2kicad:TS24CA
- added PAD17, PAD23, PAD5: PAD_T, Critbit_lib:diy_castellate_tight, symbol Connector:TestPoint
Connections:
- net BUT2 is gone; now on net LED_STA: U13.48 (MTMS/JTAG/GPIO42)
- net BOOT_BUT1: now also PAD17.1; no longer PAD2.1
- net BQ_CHG: now also U13.24 (GPIO18/ADC2_CH7); no longer U13.44 (MTCK/JTAG/GPIO39)
- net BQ_PGOOD: now also U13.27 (GPIO21); no longer U13.43 (GPIO38)
- net EN_PERIPH: now also U13.17 (GPIO12/ADC2_CH1); no longer U13.23 (GPIO17/ADC2_CH6)
- net EXTIO_1: now also U13.38 (GPIO33); no longer U13.27 (GPIO21)
- net EXTIO_2: now also U13.39 (GPIO34); no longer U13.47 (MTDI/JTAG/GPIO41)
- net EXTIO_3: now also U13.23 (GPIO17/ADC2_CH6); no longer U13.24 (GPIO18/ADC2_CH7)
- net EXTIO_7: now also U13.15 (GPIO10/ADC1_CH9); no longer U13.17 (GPIO12/ADC2_CH1)
- net GND: now also PAD5.1
- net LED_STA: no longer U13.45 (MTDO/JTAG/GPIO40)
- net PERIPH_FAULT: now also U13.47 (MTDI/JTAG/GPIO41); no longer U13.15 (GPIO10/ADC1_CH9)
- net SD_CLK: now also U13.41 (GPIO36); no longer U13.40 (GPIO35)
- net SD_CMD: now also U13.40 (GPIO35); no longer U13.38 (GPIO33)
- net SD_DAT0: now also U13.42 (GPIO37); no longer U13.41 (GPIO36)
- net SD_DAT1: now also U13.43 (GPIO38); no longer U13.42 (GPIO37)
- net SD_DET: now also U13.44 (MTCK/JTAG/GPIO39); no longer U13.39 (GPIO34)
- net WS2812_VDD: no longer R3.2
- new net: PAD23.1, R3.2
- new net EXTIO_0: PAD2.1, U13.45 (MTDO/JTAG/GPIO40)
Other:
- moved on the sheet: C17, C19, R24, R3, R5, SW1

Commit message: little schematic cleanup, add PDF and render image
Other:
- note added: "Some calculations WARN: NOT VERIFIED s3 - 2.2 s3FH8 - 3.0 c3fh4 - 1.4 c3 - 1.2 16M - 0.3-0.5 S3@8 - 3.0 S3@16 - 2.5 c3@16 - 1.5"
- note added: "WARN: Not verified Riset = 890/Itarg Itarg = 0.8A -> Riset=1.1k Itarg = 0.27A -> Riset=3k Rilim = 1550 / Itarg Iilim = 1.5A -> Rilim=1.1k Iilim = 0.5A -> Rilim=3k"
- note added: "datasheet does not specify if EP should be connected to GND, but it seems to work. other similar ICs with better datasheets recommend connecting it to GND"
- note removed: "Riset = 890/Itarg Itarg = 0.8A -> Riset=1.1k Itarg = 0.27A -> Riset=3k Rilim = 1550 / Itarg Iilim = 1.5A -> Rilim=1.1k Iilim = 0.5A -> Rilim=3k"
- note removed: "datasheet not specified if connect needed"
- note removed: "s3 - 2.2 s3FH8 - 3.0 c3fh4 - 1.4 c3 - 1.2 16M - 0.3-0.5 S3@8 - 3.0 S3@16 - 2.5 c3@16 - 1.5"
- moved on the sheet: AE1, C1, C17, C19, C2, C21, C22, C23, C24, C29, C3, C30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
